File: PSVB_EvalBoard/PSVB_EvalBoard.kicad_pcb (KiCad board)
At the start: 2 copper layers, 0 parts

Commit message: update PCB design
Parts:
- added 1V8_PWR1: 0603 1V8_PWR, LED_SMD:LED_0603_1608Metric_Pad1.05x0.95mm_HandSolder, F.Cu at (80.5, 46.0)
- added 3V3_PWR1: 0603 3V3_LED, LED_SMD:LED_0603_1608Metric_Pad1.05x0.95mm_HandSolder, F.Cu at (83.8, 46.0)
- added 5V_PWR1: 0603 5V_LED, LED_SMD:LED_0603_1608Metric_Pad1.05x0.95mm_HandSolder, F.Cu at (63.3, 34.5)
- added AKINA_JTAG1: ~, Connector_PinHeader_2.54mm:PinHeader_2x05_P2.54mm_Vertical, F.Cu at (98.4, 55.4)
- added AKINA_RESET1: KEY, Button_Switch_SMD:SW_SPST_CK_RS282G05A3, F.Cu at (202.6, 149.0)
- added BAT1: CR1220-2, zgoolib:CR1220_Holder, F.Cu at (164.6, 39.5)
- added BEEP1: BUZZER, zgoolib:BEEP_4317, F.Cu at (62.0, 151.6)
- added BOOT_MODE1: SW_SMD_2P-2.54mm, Button_Switch_SMD:SW_DIP_SPSTx02_Slide_6.7x6.64mm_W8.61mm_P2.54mm_LowProfile, F.Cu at (90.9, 116.1)
- added BOOT_MODE2: SW_SMD_2P-2.54mm, Button_Switch_SMD:SW_DIP_SPSTx02_Slide_6.7x6.64mm_W8.61mm_P2.54mm_LowProfile, F.Cu at (171.6, 130.0)
- added BTB100x1: BTB100PINx2_IC_Adapter, zgoolib:BTB100PINx2_FemaleConnector, F.Cu at (174.6, 87.7)
- added C1: 47uF, Capacitor_SMD:CP_Elec_6.3x7.7, F.Cu at (55.5, 50.2)
- added C10: 0603 4.7uF/1%, Capacitor_SMD:C_0603_1608Metric_Pad1.08x0.95mm_HandSolder, F.Cu at (93.4, 40.1)
- added C100: 0.1uF, Capacitor_SMD:C_0603_1608Metric_Pad1.08x0.95mm_HandSolder, F.Cu at (150.5, 38.6)
- added C101: 10uF, Capacitor_SMD:C_0603_1608Metric_Pad1.08x0.95mm_HandSolder, F.Cu at (152.7, 38.6)
- added C11: 0603 0.1uF/16V, Capacitor_SMD:C_0603_1608Metric_Pad1.08x0.95mm_HandSolder, F.Cu at (104.9, 45.2)
- added C12: 0603 0.1uF/16V, Capacitor_SMD:C_0603_1608Metric_Pad1.08x0.95mm_HandSolder, F.Cu at (93.2, 32.5)
- added C13: 0603 4.7uF/16V, Capacitor_SMD:C_0603_1608Metric_Pad1.08x0.95mm_HandSolder, F.Cu at (95.7, 32.5)
- added C14: 0603 0.1uF/16V, Capacitor_SMD:C_0603_1608Metric_Pad1.08x0.95mm_HandSolder, F.Cu at (105.0, 32.6)
- added C15: 0603 0.01uF/16V, Capacitor_SMD:C_0603_1608Metric_Pad1.08x0.95mm_HandSolder, F.Cu at (115.6, 32.9)
- added C16: 0603 30P/16V, Capacitor_SMD:C_0603_1608Metric_Pad1.08x0.95mm_HandSolder, F.Cu at (115.6, 36.8)
- added C17: 0603 4.7uF/1%, Capacitor_SMD:C_0603_1608Metric_Pad1.08x0.95mm_HandSolder, F.Cu at (116.0, 48.0)
- added C18: 0603 0.1uF/16V, Capacitor_SMD:C_0603_1608Metric_Pad1.08x0.95mm_HandSolder, F.Cu at (138.7, 52.8)
- added C19: 0603 0.1uF/16V, Capacitor_SMD:C_0603_1608Metric_Pad1.08x0.95mm_HandSolder, F.Cu at (138.7, 55.3)
- added C2: 22uF, Capacitor_SMD:CP_Elec_6.3x7.7, F.Cu at (55.5, 42.2)
- added C20: 0603 0.1uF/16V, Capacitor_SMD:C_0603_1608Metric_Pad1.08x0.95mm_HandSolder, F.Cu at (142.6, 53.0)
- added C21: 0603 0.1uF/16V, Capacitor_SMD:C_0603_1608Metric_Pad1.08x0.95mm_HandSolder, F.Cu at (142.6, 55.5)
- added C22: 0603 4.7uF/16V, Capacitor_SMD:C_0603_1608Metric_Pad1.08x0.95mm_HandSolder, F.Cu at (121.0, 48.4)
- added C23: 0603 0.1uF/16V, Capacitor_SMD:C_0603_1608Metric_Pad1.08x0.95mm_HandSolder, F.Cu at (123.5, 48.4)
- added C24: 0603 4.7uF/16V, Capacitor_SMD:C_0603_1608Metric_Pad1.08x0.95mm_HandSolder, F.Cu at (111.8, 48.0)
- added C25: 0603 10uF/16V, Capacitor_SMD:C_0603_1608Metric_Pad1.08x0.95mm_HandSolder, F.Cu at (147.3, 49.9)
- added C26: 0603 10uF/16V, Capacitor_SMD:C_0603_1608Metric_Pad1.08x0.95mm_HandSolder, F.Cu at (147.3, 53.1)
- added C27: 0603 10uF/16V, Capacitor_SMD:C_0603_1608Metric_Pad1.08x0.95mm_HandSolder, F.Cu at (147.3, 55.6)
- added C28: 0603 10uF/16V, Capacitor_SMD:C_0603_1608Metric_Pad1.08x0.95mm_HandSolder, F.Cu at (61.5, 64.1)
- added C29: 0603 0.1uF/16V, Capacitor_SMD:C_0603_1608Metric_Pad1.08x0.95mm_HandSolder, F.Cu at (91.3, 60.6)
- added C3: 0603 1uF/16V, Capacitor_SMD:C_0603_1608Metric_Pad1.08x0.95mm_HandSolder, F.Cu at (63.3, 45.9)
- added C30: 0603 4.7uF/16V, Capacitor_SMD:C_0603_1608Metric_Pad1.08x0.95mm_HandSolder, F.Cu at (93.8, 60.6)
- added C31: 0603 0.1uF/16V, Capacitor_SMD:C_0603_1608Metric_Pad1.08x0.95mm_HandSolder, F.Cu at (96.3, 60.6)
- added C32: 0603 4.7uF/16V, Capacitor_SMD:C_0603_1608Metric_Pad1.08x0.95mm_HandSolder, F.Cu at (98.8, 60.6)
- added C33: 0603 3.3uF/16V, Capacitor_SMD:C_0603_1608Metric_Pad1.08x0.95mm_HandSolder, F.Cu at (101.4, 60.6)
- added C34: 0603 0.1uF/16V, Capacitor_SMD:C_0603_1608Metric_Pad1.08x0.95mm_HandSolder, F.Cu at (71.2, 75.4)
- added C35: 0603 0.1uF/16V, Capacitor_SMD:C_0603_1608Metric_Pad1.08x0.95mm_HandSolder, F.Cu at (71.4, 61.7)
- added C36: 0603 27pF/16V, Capacitor_SMD:C_0603_1608Metric_Pad1.08x0.95mm_HandSolder, F.Cu at (64.6, 65.8)
- added C37: 0603 27pF/16V, Capacitor_SMD:C_0603_1608Metric_Pad1.08x0.95mm_HandSolder, F.Cu at (64.6, 68.3)
- added C38: 0.1uF, Capacitor_SMD:C_0603_1608Metric_Pad1.08x0.95mm_HandSolder, F.Cu at (80.9, 59.8)
- added C39: 0.1uF, Capacitor_SMD:C_0603_1608Metric_Pad1.08x0.95mm_HandSolder, F.Cu at (80.9, 62.3)
- added C4: 0603 1uF/16V, Capacitor_SMD:C_0603_1608Metric_Pad1.08x0.95mm_HandSolder, F.Cu at (63.3, 43.4)
- added C40: 0.1uF, Capacitor_SMD:C_0603_1608Metric_Pad1.08x0.95mm_HandSolder, F.Cu at (80.9, 64.8)
- added C41: 0.1uF, Capacitor_SMD:C_0603_1608Metric_Pad1.08x0.95mm_HandSolder, F.Cu at (86.9, 59.6)
- added C42: 0.1uF, Capacitor_SMD:C_0603_1608Metric_Pad1.08x0.95mm_HandSolder, F.Cu at (86.9, 62.1)
- added C43: 0.1uF, Capacitor_SMD:C_0603_1608Metric_Pad1.08x0.95mm_HandSolder, F.Cu at (86.9, 64.6)
- added C44: 0.1uF, Capacitor_SMD:C_0603_1608Metric_Pad1.08x0.95mm_HandSolder, F.Cu at (86.9, 67.1)
- added C45: 0603 0.1uF/16V, Capacitor_SMD:C_0603_1608Metric_Pad1.08x0.95mm_HandSolder, F.Cu at (74.4, 112.6)
- added C46: 0603 10pF/16V, Capacitor_SMD:C_0603_1608Metric_Pad1.08x0.95mm_HandSolder, F.Cu at (73.8, 96.8)
- added C47: 0603 10pF/16V, Capacitor_SMD:C_0603_1608Metric_Pad1.08x0.95mm_HandSolder, F.Cu at (73.8, 104.1)
- added C48: 0603 0.1uF/16V, Capacitor_SMD:C_0603_1608Metric_Pad1.08x0.95mm_HandSolder, F.Cu at (102.2, 86.7)
- added C49: 0.1uF, Capacitor_SMD:C_0603_1608Metric_Pad1.08x0.95mm_HandSolder, F.Cu at (74.7, 94.1)
- added C5: 0603 1uF/16V, Capacitor_SMD:C_0603_1608Metric_Pad1.08x0.95mm_HandSolder, F.Cu at (63.5, 52.1)
- added C50: 0.1uF, Capacitor_SMD:C_0603_1608Metric_Pad1.08x0.95mm_HandSolder, F.Cu at (110.6, 124.9)
- added C51: 0.1uF, Capacitor_SMD:C_0603_1608Metric_Pad1.08x0.95mm_HandSolder, F.Cu at (113.1, 124.9)
- added C52: 0.1uF, Capacitor_SMD:C_0603_1608Metric_Pad1.08x0.95mm_HandSolder, F.Cu at (115.6, 124.9)
- added C53: 0.1uF, Capacitor_SMD:C_0603_1608Metric_Pad1.08x0.95mm_HandSolder, F.Cu at (118.1, 124.9)
- added C54: 0.1uF, Capacitor_SMD:C_0603_1608Metric_Pad1.08x0.95mm_HandSolder, F.Cu at (120.6, 124.9)
- added C55: 0.1uF, Capacitor_SMD:C_0603_1608Metric_Pad1.08x0.95mm_HandSolder, F.Cu at (123.1, 124.9)
- added C56: 0.1uF, Capacitor_SMD:C_0603_1608Metric_Pad1.08x0.95mm_HandSolder, F.Cu at (125.6, 124.9)
- added C57: 0.1uF, Capacitor_SMD:C_0603_1608Metric_Pad1.08x0.95mm_HandSolder, F.Cu at (128.2, 124.9)
- added C58: 0.1uF, Capacitor_SMD:C_0603_1608Metric_Pad1.08x0.95mm_HandSolder, F.Cu at (130.7, 124.9)
- added C59: 0603 4.7uF/16V, Capacitor_SMD:C_0603_1608Metric_Pad1.08x0.95mm_HandSolder, F.Cu at (104.1, 86.7)
- added C6: 0603 1uF/16V, Capacitor_SMD:C_0603_1608Metric_Pad1.08x0.95mm_HandSolder, F.Cu at (63.5, 49.6)
- added C60: 4.7uF, Capacitor_SMD:C_0603_1608Metric_Pad1.08x0.95mm_HandSolder, F.Cu at (72.8, 94.1)
- added C61: 4.7uF, Capacitor_SMD:C_0603_1608Metric_Pad1.08x0.95mm_HandSolder, F.Cu at (110.1, 129.1)
- added C62: 4.7uF, Capacitor_SMD:C_0603_1608Metric_Pad1.08x0.95mm_HandSolder, F.Cu at (112.6, 129.1)
- added C63: 4.7uF, Capacitor_SMD:C_0603_1608Metric_Pad1.08x0.95mm_HandSolder, F.Cu at (115.2, 129.1)
- added C64: 4.7uF, Capacitor_SMD:C_0603_1608Metric_Pad1.08x0.95mm_HandSolder, F.Cu at (117.7, 129.1)
- added C65: 4.7uF, Capacitor_SMD:C_0603_1608Metric_Pad1.08x0.95mm_HandSolder, F.Cu at (120.2, 129.1)
- added C67: 4.7uF, Capacitor_SMD:C_0603_1608Metric_Pad1.08x0.95mm_HandSolder, F.Cu at (122.7, 129.1)
- added C68: 4.7uF, Capacitor_SMD:C_0603_1608Metric_Pad1.08x0.95mm_HandSolder, F.Cu at (125.2, 129.1)
- added C69: 4.7uF, Capacitor_SMD:C_0603_1608Metric_Pad1.08x0.95mm_HandSolder, F.Cu at (127.7, 129.1)
- added C7: 0603 1uF/16V, Capacitor_SMD:C_0603_1608Metric_Pad1.08x0.95mm_HandSolder, F.Cu at (66.4, 35.5)
- added C70: 4.7uF, Capacitor_SMD:C_0603_1608Metric_Pad1.08x0.95mm_HandSolder, F.Cu at (130.2, 129.1)
- added C71: 0603 0.1uF/16V, Capacitor_SMD:C_0603_1608Metric_Pad1.08x0.95mm_HandSolder, F.Cu at (102.7, 117.4)
- added C72: 0603 0.1uF/16V, Capacitor_SMD:C_0603_1608Metric_Pad1.08x0.95mm_HandSolder, F.Cu at (102.7, 119.9)
- added C73: 0603 20PF/16V, Capacitor_SMD:C_0603_1608Metric_Pad1.08x0.95mm_HandSolder, F.Cu at (147.7, 123.8)
- added C74: 0603 20PF/16V, Capacitor_SMD:C_0603_1608Metric_Pad1.08x0.95mm_HandSolder, F.Cu at (147.7, 126.3)
- added C75: 0603 0.1uF/16V, Capacitor_SMD:C_0603_1608Metric_Pad1.08x0.95mm_HandSolder, F.Cu at (153.2, 142.7)
- added C76: 0603 20PF/16V, Capacitor_SMD:C_0603_1608Metric_Pad1.08x0.95mm_HandSolder, F.Cu at (77.0, 132.1)
- added C77: 0603 20PF/16V, Capacitor_SMD:C_0603_1608Metric_Pad1.08x0.95mm_HandSolder, F.Cu at (77.0, 134.6)
- added C78: 0603 0.1uF/16V, Capacitor_SMD:C_0603_1608Metric_Pad1.08x0.95mm_HandSolder, F.Cu at (94.2, 134.6)
- added C79: 0603 0.1uF/16V, Capacitor_SMD:C_0603_1608Metric_Pad1.08x0.95mm_HandSolder, F.Cu at (204.5, 141.9)
- added C8: 0603 1uF/16V, Capacitor_SMD:C_0603_1608Metric_Pad1.08x0.95mm_HandSolder, F.Cu at (85.2, 35.5)
- added C80: 0.1uF, Capacitor_SMD:C_0603_1608Metric_Pad1.08x0.95mm_HandSolder, F.Cu at (178.1, 87.8)
- added C81: 0.1uF, Capacitor_SMD:C_0603_1608Metric_Pad1.08x0.95mm_HandSolder, F.Cu at (175.6, 87.8)
- added C82: 0.01uF, Capacitor_SMD:C_0603_1608Metric_Pad1.08x0.95mm_HandSolder, F.Cu at (166.4, 72.8)
- added C83: 2.2nF, Capacitor_SMD:C_0603_1608Metric_Pad1.08x0.95mm_HandSolder, F.Cu at (168.9, 72.8)
- added C84: 0.1uF, Capacitor_SMD:C_0603_1608Metric_Pad1.08x0.95mm_HandSolder, F.Cu at (171.4, 72.8)
- added C85: 0.1uF, Capacitor_SMD:C_0603_1608Metric_Pad1.08x0.95mm_HandSolder, F.Cu at (173.9, 72.8)
- added C86: 0.1uF, Capacitor_SMD:C_0603_1608Metric_Pad1.08x0.95mm_HandSolder, F.Cu at (177.9, 96.9)
- added C87: 0.1uF, Capacitor_SMD:C_0603_1608Metric_Pad1.08x0.95mm_HandSolder, F.Cu at (177.9, 99.4)
- added C88: 0.1uF, Capacitor_SMD:C_0603_1608Metric_Pad1.08x0.95mm_HandSolder, F.Cu at (178.7, 38.7)
- added C89: 0.1uF, Capacitor_SMD:C_0603_1608Metric_Pad1.08x0.95mm_HandSolder, F.Cu at (178.7, 35.5)
- added C9: 0603 0.1uF/1%, Capacitor_SMD:C_0603_1608Metric_Pad1.08x0.95mm_HandSolder, F.Cu at (90.9, 40.1)
- added C90: 0.1uF, Capacitor_SMD:C_0603_1608Metric_Pad1.08x0.95mm_HandSolder, F.Cu at (188.1, 38.7)
- added C91: 0.1uF, Capacitor_SMD:C_0603_1608Metric_Pad1.08x0.95mm_HandSolder, F.Cu at (188.1, 35.6)
- added C92: 0.1uF, Capacitor_SMD:C_0603_1608Metric_Pad1.08x0.95mm_HandSolder, F.Cu at (197.5, 38.4)
- added C93: 0.1uF, Capacitor_SMD:C_0603_1608Metric_Pad1.08x0.95mm_HandSolder, F.Cu at (197.5, 35.4)
- added C94: 0.1uF, Capacitor_SMD:C_0603_1608Metric_Pad1.08x0.95mm_HandSolder, F.Cu at (206.9, 38.4)
- added C95: 0.1uF, Capacitor_SMD:C_0603_1608Metric_Pad1.08x0.95mm_HandSolder, F.Cu at (206.9, 35.4)
- added C96: 0.1uF, Capacitor_SMD:C_0603_1608Metric_Pad1.08x0.95mm_HandSolder, F.Cu at (109.5, 101.7)
- added C97: 0.1uF, Capacitor_SMD:C_0603_1608Metric_Pad1.08x0.95mm_HandSolder, F.Cu at (232.5, 91.5)
- added C98: 0.1uF, Capacitor_SMD:C_0603_1608Metric_Pad1.08x0.95mm_HandSolder, F.Cu at (235.0, 91.5)
- added C99: 0.1uF, Capacitor_SMD:C_0603_1608Metric_Pad1.08x0.95mm_HandSolder, F.Cu at (237.6, 91.5)
- added D1: 1N4148, Diode_SMD:D_SOD-123, F.Cu at (71.0, 151.5)
- added ESD1: SD24C-TP, Diode_SMD:D_SOD-323_HandSoldering, F.Cu at (63.9, 73.2)
- added ESD2: SD24C-TP, Diode_SMD:D_SOD-323_HandSoldering, F.Cu at (64.0, 78.7)
- added ESD3: SD24C-TP, Diode_SMD:D_SOD-323_HandSoldering, F.Cu at (64.2, 86.7)
- added ESD4: SD24C-TP, Diode_SMD:D_SOD-323_HandSoldering, F.Cu at (64.2, 91.6)
- added ETH1: HR911105A, zgoolib:RJ45_HanRun_HR911105A, F.Cu at (130.3, 137.7)
- added ETH2: HR911105A, zgoolib:RJ45_HanRun_HR911105A, F.Cu at (100.5, 137.7)
- added F1: 1206 10V/2A, Fuse:Fuse_1206_3216Metric_Pad1.42x1.75mm_HandSolder, F.Cu at (60.2, 57.3)
- added J1: ~, Connector_PinHeader_2.54mm:PinHeader_2x04_P2.54mm_Vertical, F.Cu at (140.2, 34.0)
- added J10: PIN20, Connector_PinHeader_2.54mm:PinHeader_2x10_P2.54mm_Vertical, F.Cu at (124.4, 88.9)
- added J11: PIN12_2x6, Connector_PinHeader_2.54mm:PinHeader_2x06_P2.54mm_Vertical, F.Cu at (129.4, 119.4)
- added J12: PIN20, Connector_PinHeader_2.54mm:PinHeader_2x10_P2.54mm_Vertical, F.Cu at (236.3, 82.2)
- added J13: PIN6_2x3, Connector_PinHeader_2.54mm:PinHeader_2x03_P2.54mm_Vertical, F.Cu at (236.4, 100.8)
- added J14: ~, Connector_PinHeader_2.54mm:PinHeader_1x04_P2.54mm_Vertical, F.Cu at (220.0, 33.8)
- added J15: ~, Connector_PinHeader_2.54mm:PinHeader_1x04_P2.54mm_Vertical, F.Cu at (228.3, 33.7)
- added J16: ~, Connector_PinHeader_2.54mm:PinHeader_1x04_P2.54mm_Vertical, F.Cu at (228.3, 46.0)
- added J17: ~, Connector_PinHeader_2.54mm:PinHeader_1x04_P2.54mm_Vertical, F.Cu at (220.0, 46.4)
- added J18: ~, Connector_PinHeader_2.54mm:PinHeader_1x04_P2.54mm_Vertical, F.Cu at (236.3, 46.0)
- added J19: ~, Connector_PinHeader_2.54mm:PinHeader_2x04_P2.54mm_Vertical, F.Cu at (209.7, 46.5)
- added J2: PIN2, Connector_PinHeader_2.54mm:PinHeader_1x02_P2.54mm_Vertical, F.Cu at (53.0, 68.8)
- added J20: ~, Connector_PinHeader_2.54mm:PinHeader_1x06_P2.54mm_Vertical, F.Cu at (224.3, 119.4)
- added J21: ~, Connector_PinHeader_2.54mm:PinHeader_1x06_P2.54mm_Vertical, F.Cu at (224.3, 126.4)
- added J22: ~, Connector_PinHeader_2.54mm:PinHeader_1x06_P2.54mm_Vertical, F.Cu at (224.3, 133.3)
- added J23: ~, Connector_PinHeader_2.54mm:PinHeader_1x06_P2.54mm_Vertical, F.Cu at (224.3, 140.3)
- added J24: ~, Connector_PinHeader_2.54mm:PinHeader_1x03_P2.54mm_Vertical, F.Cu at (184.3, 33.8)
- added J25: ~, Connector_PinHeader_2.54mm:PinHeader_1x03_P2.54mm_Vertical, F.Cu at (193.7, 33.8)
- added J26: ~, Connector_PinHeader_2.54mm:PinHeader_1x03_P2.54mm_Vertical, F.Cu at (203.1, 33.7)
- added J27: ~, Connector_PinHeader_2.54mm:PinHeader_1x03_P2.54mm_Vertical, F.Cu at (212.5, 33.8)
- added J28: ~, Connector_PinHeader_2.54mm:PinHeader_1x03_P2.54mm_Vertical, F.Cu at (106.6, 96.6)
- added J29: PIN6_2x3, Connector_PinHeader_2.54mm:PinHeader_2x03_P2.54mm_Vertical, F.Cu at (106.9, 66.1)
- added J3: PIN20, Connector_PinHeader_2.54mm:PinHeader_2x10_P2.54mm_Vertical, F.Cu at (53.7, 99.9)
- added J30: PIN6_2x3, Connector_PinHeader_2.54mm:PinHeader_2x03_P2.54mm_Vertical, F.Cu at (107.4, 83.8)
- added J31: PIN6_2x3, Connector_PinHeader_2.54mm:PinHeader_2x03_P2.54mm_Vertical, F.Cu at (117.4, 151.8)
- added J4: PIN20, Connector_PinHeader_2.54mm:PinHeader_2x10_P2.54mm_Vertical, F.Cu at (116.7, 119.4)
- added J5: PIN20, Connector_PinHeader_2.54mm:PinHeader_2x10_P2.54mm_Vertical, F.Cu at (63.0, 99.9)
- added J6: PIN20, Connector_PinHeader_2.54mm:PinHeader_2x10_P2.54mm_Vertical, F.Cu at (116.7, 88.9)
- added J7: PIN20, Connector_PinHeader_2.54mm:PinHeader_2x10_P2.54mm_Vertical, F.Cu at (228.2, 82.2)
- added J8: PIN20, Connector_PinHeader_2.54mm:PinHeader_2x10_P2.54mm_Vertical, F.Cu at (228.1, 110.2)
- added J9: PIN20, Connector_PinHeader_2.54mm:PinHeader_2x10_P2.54mm_Vertical, F.Cu at (124.4, 119.4)
- added KEY1: SW_Push, Button_Switch_SMD:SW_SPST_CK_RS282G05A3, F.Cu at (176.4, 149.2)
- added KEY2: SW_Push, Button_Switch_SMD:SW_SPST_CK_RS282G05A3, F.Cu at (181.6, 149.2)
- added KEY3: SW_Push, Button_Switch_SMD:SW_SPST_CK_RS282G05A3, F.Cu at (186.7, 149.2)
- added KEY4: SW_Push, Button_Switch_SMD:SW_SPST_CK_RS282G05A3, F.Cu at (191.9, 149.2)
- added KEY5: 5Axises_KEY, zgoolib:5Axises_Key, F.Cu at (218.4, 149.1)
- added KEY6: SW_Push, Button_Switch_SMD:SW_SPST_CK_RS282G05A3, F.Cu at (151.2, 149.2)
- added KEY7: SW_Push, Button_Switch_SMD:SW_SPST_CK_RS282G05A3, F.Cu at (156.3, 149.2)
- added KEY8: SW_Push, Button_Switch_SMD:SW_SPST_CK_RS282G05A3, F.Cu at (161.5, 149.2)
- added KEY9: SW_Push, Button_Switch_SMD:SW_SPST_CK_RS282G05A3, F.Cu at (166.6, 149.2)
- added L1: 2.2uH/1A, zgoolib:SWPA3010, F.Cu at (80.6, 34.7)
- added L2: 6.8nH/500mA, Inductor_SMD:L_0603_1608Metric_Pad1.05x0.95mm_HandSolder, F.Cu at (59.6, 64.1)
- added L3: 6.8nH/500mA, Inductor_SMD:L_0603_1608Metric_Pad1.05x0.95mm_HandSolder, F.Cu at (65.2, 56.3)
- added L4: 6.8nH/500mA, Inductor_SMD:L_0603_1608Metric_Pad1.05x0.95mm_HandSolder, F.Cu at (65.2, 58.8)
- added LED1: YELLOW, LED_SMD:LED_0603_1608Metric_Pad1.05x0.95mm_HandSolder, F.Cu at (185.2, 136.3)
- added LED10: LD271, LED_SMD:LED_0603_1608Metric_Pad1.05x0.95mm_HandSolder, F.Cu at (71.2, 145.7)
- added LED11: LD271, LED_SMD:LED_0603_1608Metric_Pad1.05x0.95mm_HandSolder, F.Cu at (74.2, 145.7)
- added LED12: LD271, LED_SMD:LED_0603_1608Metric_Pad1.05x0.95mm_HandSolder, F.Cu at (77.2, 145.7)
- added LED2: YELLOW, LED_SMD:LED_0603_1608Metric_Pad1.05x0.95mm_HandSolder, F.Cu at (188.3, 136.3)
- added LED3: LD271, LED_SMD:LED_0603_1608Metric_Pad1.05x0.95mm_HandSolder, F.Cu at (191.4, 136.3)
- added LED4: LD271, LED_SMD:LED_0603_1608Metric_Pad1.05x0.95mm_HandSolder, F.Cu at (194.4, 136.3)
- added LED5: LD271, LED_SMD:LED_0603_1608Metric_Pad1.05x0.95mm_HandSolder, F.Cu at (197.5, 136.3)
- added LED6: LD271, LED_SMD:LED_0603_1608Metric_Pad1.05x0.95mm_HandSolder, F.Cu at (200.5, 136.3)
- added LED7: LD271, LED_SMD:LED_0603_1608Metric_Pad1.05x0.95mm_HandSolder, F.Cu at (203.6, 136.3)
- added LED8: LD271, LED_SMD:LED_0603_1608Metric_Pad1.05x0.95mm_HandSolder, F.Cu at (206.6, 136.3)
- added LED9: LD271, LED_SMD:LED_0603_1608Metric_Pad1.05x0.95mm_HandSolder, F.Cu at (68.1, 145.7)
- added POWER1: SW_SELF_LOCK_5.8mm-5.8mm-10mm, zgoolib:SelfLock_Switch, F.Cu at (54.6, 60.3)
- added Q1: S9013, Package_TO_SOT_SMD:SOT-23, F.Cu at (67.2, 150.9)
- added R1: 0603 5K/1%, Resistor_SMD:R_0603_1608Metric_Pad0.98x0.95mm_HandSolder, F.Cu at (63.3, 36.5)
- added R10: 0603 0R/1%, Resistor_SMD:R_0603_1608Metric_Pad0.98x0.95mm_HandSolder, F.Cu at (96.3, 40.1)
- added R100: 0R/1%, Resistor_SMD:R_0603_1608Metric_Pad0.98x0.95mm_HandSolder, F.Cu at (217.2, 33.7)
- added R101: 0R/1%, Resistor_SMD:R_0603_1608Metric_Pad0.98x0.95mm_HandSolder, F.Cu at (217.2, 41.5)
- added R102: 0R/1%, Resistor_SMD:R_0603_1608Metric_Pad0.98x0.95mm_HandSolder, F.Cu at (225.6, 33.5)
- added R103: 0R/1%, Resistor_SMD:R_0603_1608Metric_Pad0.98x0.95mm_HandSolder, F.Cu at (225.6, 41.4)
- added R104: 0R/1%, Resistor_SMD:R_0603_1608Metric_Pad0.98x0.95mm_HandSolder, F.Cu at (225.6, 45.9)
- added R105: 0R/1%, Resistor_SMD:R_0603_1608Metric_Pad0.98x0.95mm_HandSolder, F.Cu at (225.6, 53.7)
- added R106: 0R/1%, Resistor_SMD:R_0603_1608Metric_Pad0.98x0.95mm_HandSolder, F.Cu at (217.2, 46.2)
- added R107: 0R/1%, Resistor_SMD:R_0603_1608Metric_Pad0.98x0.95mm_HandSolder, F.Cu at (217.2, 54.1)
- added R108: 0R/1%, Resistor_SMD:R_0603_1608Metric_Pad0.98x0.95mm_HandSolder, F.Cu at (233.6, 45.9)
- added R109: 0R/1%, Resistor_SMD:R_0603_1608Metric_Pad0.98x0.95mm_HandSolder, F.Cu at (233.6, 53.7)
- added R11: 0603 0R/1%, Resistor_SMD:R_0603_1608Metric_Pad0.98x0.95mm_HandSolder, F.Cu at (98.8, 40.1)
- added R110: 0R/1%, Resistor_SMD:R_0603_1608Metric_Pad0.98x0.95mm_HandSolder, F.Cu at (224.2, 116.6)
- added R111: 0R/1%, Resistor_SMD:R_0603_1608Metric_Pad0.98x0.95mm_HandSolder, F.Cu at (229.5, 116.6)
- added R112: 0R/1%, Resistor_SMD:R_0603_1608Metric_Pad0.98x0.95mm_HandSolder, F.Cu at (234.8, 116.6)
- added R113: 0R/1%, Resistor_SMD:R_0603_1608Metric_Pad0.98x0.95mm_HandSolder, F.Cu at (224.2, 123.6)
- added R114: 0R/1%, Resistor_SMD:R_0603_1608Metric_Pad0.98x0.95mm_HandSolder, F.Cu at (228.5, 123.6)
- added R115: 0R/1%, Resistor_SMD:R_0603_1608Metric_Pad0.98x0.95mm_HandSolder, F.Cu at (232.9, 123.6)
- added R116: 0R/1%, Resistor_SMD:R_0603_1608Metric_Pad0.98x0.95mm_HandSolder, F.Cu at (237.1, 123.6)
- added R117: 0R/1%, Resistor_SMD:R_0603_1608Metric_Pad0.98x0.95mm_HandSolder, F.Cu at (224.2, 130.6)
- added R118: 0R/1%, Resistor_SMD:R_0603_1608Metric_Pad0.98x0.95mm_HandSolder, F.Cu at (229.6, 130.6)
- added R119: 0R/1%, Resistor_SMD:R_0603_1608Metric_Pad0.98x0.95mm_HandSolder, F.Cu at (234.9, 130.6)
- added R12: 0603 0R/1%, Resistor_SMD:R_0603_1608Metric_Pad0.98x0.95mm_HandSolder, F.Cu at (104.9, 42.2)
- added R120: 0R/1%, Resistor_SMD:R_0603_1608Metric_Pad0.98x0.95mm_HandSolder, F.Cu at (224.2, 137.5)
- added R121: 0R/1%, Resistor_SMD:R_0603_1608Metric_Pad0.98x0.95mm_HandSolder, F.Cu at (229.6, 137.5)
- added R122: 0R/1%, Resistor_SMD:R_0603_1608Metric_Pad0.98x0.95mm_HandSolder, F.Cu at (234.9, 137.5)
- added R123: 10K/1%, Resistor_SMD:R_0603_1608Metric_Pad0.98x0.95mm_HandSolder, F.Cu at (178.7, 32.4)
- added R124: 10K/1%, Resistor_SMD:R_0603_1608Metric_Pad0.98x0.95mm_HandSolder, F.Cu at (181.5, 36.4)
- added R125: 10K/1%, Resistor_SMD:R_0603_1608Metric_Pad0.98x0.95mm_HandSolder, F.Cu at (188.1, 32.4)
- added R126: 10K/1%, Resistor_SMD:R_0603_1608Metric_Pad0.98x0.95mm_HandSolder, F.Cu at (190.9, 36.4)
- added R127: 10K/1%, Resistor_SMD:R_0603_1608Metric_Pad0.98x0.95mm_HandSolder, F.Cu at (197.5, 32.4)
- added R128: 10K/1%, Resistor_SMD:R_0603_1608Metric_Pad0.98x0.95mm_HandSolder, F.Cu at (200.3, 36.3)
- added R129: 10K/1%, Resistor_SMD:R_0603_1608Metric_Pad0.98x0.95mm_HandSolder, F.Cu at (206.9, 32.4)
- added R13: 0603 0R/1%, Resistor_SMD:R_0603_1608Metric_Pad0.98x0.95mm_HandSolder, F.Cu at (100.3, 32.5)
- added R130: 10K/1%, Resistor_SMD:R_0603_1608Metric_Pad0.98x0.95mm_HandSolder, F.Cu at (209.7, 36.3)
- added R131: 0603 100R/1%, Resistor_SMD:R_0603_1608Metric_Pad0.98x0.95mm_HandSolder, F.Cu at (109.5, 96.4)
- added R132: 0R/1%, Resistor_SMD:R_0603_1608Metric_Pad0.98x0.95mm_HandSolder, F.Cu at (68.2, 87.9)
- added R133: 0R/1%, Resistor_SMD:R_0603_1608Metric_Pad0.98x0.95mm_HandSolder, F.Cu at (68.2, 90.3)
- added R134: 0603 1K/1%, Resistor_SMD:R_0603_1608Metric_Pad0.98x0.95mm_HandSolder, F.Cu at (68.2, 141.0)
- added R135: 0603 1K/1%, Resistor_SMD:R_0603_1608Metric_Pad0.98x0.95mm_HandSolder, F.Cu at (70.7, 141.0)
- added R136: 0603 1K/1%, Resistor_SMD:R_0603_1608Metric_Pad0.98x0.95mm_HandSolder, F.Cu at (73.2, 141.0)
- added R137: 0603 1K/1%, Resistor_SMD:R_0603_1608Metric_Pad0.98x0.95mm_HandSolder, F.Cu at (75.8, 141.0)
- added R138: 0603 1K/1%, Resistor_SMD:R_0603_1608Metric_Pad0.98x0.95mm_HandSolder, F.Cu at (74.5, 150.7)
- added R139: 0603 10K/1%, Resistor_SMD:R_0603_1608Metric_Pad0.98x0.95mm_HandSolder, F.Cu at (74.5, 153.2)
- added R14: 0603 0R/1%, Resistor_SMD:R_0603_1608Metric_Pad0.98x0.95mm_HandSolder, F.Cu at (97.8, 32.5)
- added R140: 0603 10K/1%, Resistor_SMD:R_0603_1608Metric_Pad0.98x0.95mm_HandSolder, F.Cu at (162.1, 141.4)
- added R141: 0603 10K/1%, Resistor_SMD:R_0603_1608Metric_Pad0.98x0.95mm_HandSolder, F.Cu at (164.6, 141.4)
- added R142: 0603 10K/1%, Resistor_SMD:R_0603_1608Metric_Pad0.98x0.95mm_HandSolder, F.Cu at (167.1, 141.4)
- added R143: 0603 10K/1%, Resistor_SMD:R_0603_1608Metric_Pad0.98x0.95mm_HandSolder, F.Cu at (169.6, 141.4)
- added R144: 0603 10K/1%, Resistor_SMD:R_0603_1608Metric_Pad0.98x0.95mm_HandSolder, F.Cu at (200.2, 97.2)
- added R145: 0603 10K/1%, Resistor_SMD:R_0603_1608Metric_Pad0.98x0.95mm_HandSolder, F.Cu at (200.2, 99.7)
- added R146: 0603 10K/1%, Resistor_SMD:R_0603_1608Metric_Pad0.98x0.95mm_HandSolder, F.Cu at (200.2, 102.2)
- added R147: 0603 10K/1%, Resistor_SMD:R_0603_1608Metric_Pad0.98x0.95mm_HandSolder, F.Cu at (200.2, 104.7)
- added R148: 0603 10K/1%, Resistor_SMD:R_0603_1608Metric_Pad0.98x0.95mm_HandSolder, F.Cu at (200.2, 107.2)
- added R149: 0603 10K/1%, Resistor_SMD:R_0603_1608Metric_Pad0.98x0.95mm_HandSolder, F.Cu at (218.3, 97.8)
- added R15: 0603 0R/1%, Resistor_SMD:R_0603_1608Metric_Pad0.98x0.95mm_HandSolder, F.Cu at (104.9, 35.3)
- added R150: 0603 10K/1%, Resistor_SMD:R_0603_1608Metric_Pad0.98x0.95mm_HandSolder, F.Cu at (218.3, 95.2)
- added R151: 0603 10K/1%, Resistor_SMD:R_0603_1608Metric_Pad0.98x0.95mm_HandSolder, F.Cu at (218.3, 92.7)
- added R152: 0603 10K/1%, Resistor_SMD:R_0603_1608Metric_Pad0.98x0.95mm_HandSolder, F.Cu at (218.3, 90.2)
- added R153: 0603 10K/1%, Resistor_SMD:R_0603_1608Metric_Pad0.98x0.95mm_HandSolder, F.Cu at (218.3, 87.7)
- added R154: 0603 10K/1%, Resistor_SMD:R_0603_1608Metric_Pad0.98x0.95mm_HandSolder, F.Cu at (218.3, 84.1)
- added R155: 0603 10K/1%, Resistor_SMD:R_0603_1608Metric_Pad0.98x0.95mm_HandSolder, F.Cu at (218.4, 80.9)
- added R156: 0603 10K/1%, Resistor_SMD:R_0603_1608Metric_Pad0.98x0.95mm_HandSolder, F.Cu at (218.4, 78.4)
- added R157: 0603 10K/1%, Resistor_SMD:R_0603_1608Metric_Pad0.98x0.95mm_HandSolder, F.Cu at (218.4, 75.9)
- added R158: 0603 10K/1%, Resistor_SMD:R_0603_1608Metric_Pad0.98x0.95mm_HandSolder, F.Cu at (218.4, 73.4)
- added R159: 0603 10K/1%, Resistor_SMD:R_0603_1608Metric_Pad0.98x0.95mm_HandSolder, F.Cu at (218.4, 70.9)
- added R16: 0603 10K/1%, Resistor_SMD:R_0603_1608Metric_Pad0.98x0.95mm_HandSolder, F.Cu at (116.0, 50.7)
- added R160: 0603 10K/1%, Resistor_SMD:R_0603_1608Metric_Pad0.98x0.95mm_HandSolder, F.Cu at (195.8, 94.3)
- added R161: 0603 10K/1%, Resistor_SMD:R_0603_1608Metric_Pad0.98x0.95mm_HandSolder, F.Cu at (195.8, 91.8)
- added R162: 0603 10K/1%, Resistor_SMD:R_0603_1608Metric_Pad0.98x0.95mm_HandSolder, F.Cu at (195.8, 89.3)
- added R164: 0603 10K/1%, Resistor_SMD:R_0603_1608Metric_Pad0.98x0.95mm_HandSolder, F.Cu at (195.8, 86.8)
- added R165: 0603 10K/1%, Resistor_SMD:R_0603_1608Metric_Pad0.98x0.95mm_HandSolder, F.Cu at (195.8, 84.3)
- added R166: 0603 10K/1%, Resistor_SMD:R_0603_1608Metric_Pad0.98x0.95mm_HandSolder, F.Cu at (195.8, 81.8)
- added R167: 0603 10K/1%, Resistor_SMD:R_0603_1608Metric_Pad0.98x0.95mm_HandSolder, F.Cu at (195.8, 79.2)
- added R168: 0603 10K/1%, Resistor_SMD:R_0603_1608Metric_Pad0.98x0.95mm_HandSolder, F.Cu at (195.8, 76.7)
- added R169: 0603 10K/1%, Resistor_SMD:R_0603_1608Metric_Pad0.98x0.95mm_HandSolder, F.Cu at (195.8, 74.2)
- added R17: 0603 0R/1%, Resistor_SMD:R_0603_1608Metric_Pad0.98x0.95mm_HandSolder, F.Cu at (138.8, 46.5)
- added R170: 0603 10K/1%, Resistor_SMD:R_0603_1608Metric_Pad0.98x0.95mm_HandSolder, F.Cu at (195.8, 106.3)
- added R171: 0603 10K/1%, Resistor_SMD:R_0603_1608Metric_Pad0.98x0.95mm_HandSolder, F.Cu at (195.8, 103.8)
- added R172: 0603 10K/1%, Resistor_SMD:R_0603_1608Metric_Pad0.98x0.95mm_HandSolder, F.Cu at (195.8, 101.3)
- added R173: 0603 10K/1%, Resistor_SMD:R_0603_1608Metric_Pad0.98x0.95mm_HandSolder, F.Cu at (147.2, 107.7)
- added R174: 0603 10K/1%, Resistor_SMD:R_0603_1608Metric_Pad0.98x0.95mm_HandSolder, F.Cu at (147.2, 105.2)
- added R175: 0603 10K/1%, Resistor_SMD:R_0603_1608Metric_Pad0.98x0.95mm_HandSolder, F.Cu at (147.2, 102.7)
- added R176: 0603 10K/1%, Resistor_SMD:R_0603_1608Metric_Pad0.98x0.95mm_HandSolder, F.Cu at (147.2, 100.2)
- added R177: 0603 10K/1%, Resistor_SMD:R_0603_1608Metric_Pad0.98x0.95mm_HandSolder, F.Cu at (147.2, 97.2)
- added R178: 0603 10K/1%, Resistor_SMD:R_0603_1608Metric_Pad0.98x0.95mm_HandSolder, F.Cu at (130.9, 102.5)
- added R179: 0603 10K/1%, Resistor_SMD:R_0603_1608Metric_Pad0.98x0.95mm_HandSolder, F.Cu at (130.9, 100.0)
- added R18: 0603 0R/1%, Resistor_SMD:R_0603_1608Metric_Pad0.98x0.95mm_HandSolder, F.Cu at (138.7, 49.0)
- added R180: 0603 10K/1%, Resistor_SMD:R_0603_1608Metric_Pad0.98x0.95mm_HandSolder, F.Cu at (131.2, 85.5)
- added R181: 0603 10K/1%, Resistor_SMD:R_0603_1608Metric_Pad0.98x0.95mm_HandSolder, F.Cu at (131.1, 82.4)
- added R183: 0603 10K/1%, Resistor_SMD:R_0603_1608Metric_Pad0.98x0.95mm_HandSolder, F.Cu at (131.1, 79.2)
- added R184: 0603 10K/1%, Resistor_SMD:R_0603_1608Metric_Pad0.98x0.95mm_HandSolder, F.Cu at (131.1, 75.9)
- added R185: 0603 10K/1%, Resistor_SMD:R_0603_1608Metric_Pad0.98x0.95mm_HandSolder, F.Cu at (130.9, 72.5)
- added R186: 0603 10K/1%, Resistor_SMD:R_0603_1608Metric_Pad0.98x0.95mm_HandSolder, F.Cu at (131.1, 69.3)
- added R187: 0603 10K/1%, Resistor_SMD:R_0603_1608Metric_Pad0.98x0.95mm_HandSolder, F.Cu at (131.2, 66.2)
- added R188: 0603 10K/1%, Resistor_SMD:R_0603_1608Metric_Pad0.98x0.95mm_HandSolder, F.Cu at (130.9, 96.9)
- added R189: 0603 10K/1%, Resistor_SMD:R_0603_1608Metric_Pad0.98x0.95mm_HandSolder, F.Cu at (130.9, 93.9)
- added R19: 0603 0R/1%, Resistor_SMD:R_0603_1608Metric_Pad0.98x0.95mm_HandSolder, F.Cu at (138.7, 51.0)
- added R190: 0603 10K/1%, Resistor_SMD:R_0603_1608Metric_Pad0.98x0.95mm_HandSolder, F.Cu at (130.9, 90.7)
- added R191: 0603 10K/1%, Resistor_SMD:R_0603_1608Metric_Pad0.98x0.95mm_HandSolder, F.Cu at (135.5, 113.8)
- added R192: 0603 10K/1%, Resistor_SMD:R_0603_1608Metric_Pad0.98x0.95mm_HandSolder, F.Cu at (130.7, 113.5)
- added R193: 0603 10K/1%, Resistor_SMD:R_0603_1608Metric_Pad0.98x0.95mm_HandSolder, F.Cu at (130.7, 110.5)
- added R194: 0603 10K/1%, Resistor_SMD:R_0603_1608Metric_Pad0.98x0.95mm_HandSolder, F.Cu at (130.7, 108.0)
- added R195: 0603 10K/1%, Resistor_SMD:R_0603_1608Metric_Pad0.98x0.95mm_HandSolder, F.Cu at (130.7, 105.5)
- added R196: 0603 10K/1%, Resistor_SMD:R_0603_1608Metric_Pad0.98x0.95mm_HandSolder, F.Cu at (147.3, 82.9)
- added R197: 0603 10K/1%, Resistor_SMD:R_0603_1608Metric_Pad0.98x0.95mm_HandSolder, F.Cu at (147.3, 85.4)
- added R2: 0603 1K/1%, Resistor_SMD:R_0603_1608Metric_Pad0.98x0.95mm_HandSolder, F.Cu at (80.5, 39.4)
- added R20: 0603 0R/1%, Resistor_SMD:R_0603_1608Metric_Pad0.98x0.95mm_HandSolder, F.Cu at (142.6, 46.2)
- added R203: 0603 10K/1%, Resistor_SMD:R_0603_1608Metric_Pad0.98x0.95mm_HandSolder, F.Cu at (147.3, 87.9)
- added R204: 0603 10K/1%, Resistor_SMD:R_0603_1608Metric_Pad0.98x0.95mm_HandSolder, F.Cu at (147.3, 90.4)
- added R205: 0603 10K/1%, Resistor_SMD:R_0603_1608Metric_Pad0.98x0.95mm_HandSolder, F.Cu at (147.3, 92.9)
- added R207: 0603 10K/1%, Resistor_SMD:R_0603_1608Metric_Pad0.98x0.95mm_HandSolder, F.Cu at (147.3, 95.4)
- added R208: 0603 10K/1%, Resistor_SMD:R_0603_1608Metric_Pad0.98x0.95mm_HandSolder, F.Cu at (153.2, 87.5)
- added R21: 0603 0R/1%, Resistor_SMD:R_0603_1608Metric_Pad0.98x0.95mm_HandSolder, F.Cu at (142.6, 48.7)
- added R213: 0603 10K/1%, Resistor_SMD:R_0603_1608Metric_Pad0.98x0.95mm_HandSolder, F.Cu at (153.2, 85.0)
- added R214: 0603 10K/1%, Resistor_SMD:R_0603_1608Metric_Pad0.98x0.95mm_HandSolder, F.Cu at (153.2, 82.5)
- added R215: 0603 10K/1%, Resistor_SMD:R_0603_1608Metric_Pad0.98x0.95mm_HandSolder, F.Cu at (153.2, 80.0)
- added R216: 0603 10K/1%, Resistor_SMD:R_0603_1608Metric_Pad0.98x0.95mm_HandSolder, F.Cu at (153.2, 77.5)
- added R217: 0603 10K/1%, Resistor_SMD:R_0603_1608Metric_Pad0.98x0.95mm_HandSolder, F.Cu at (153.2, 75.0)
- added R218: 0603 10K/1%, Resistor_SMD:R_0603_1608Metric_Pad0.98x0.95mm_HandSolder, F.Cu at (153.2, 72.5)
- added R219: 0603 10K/1%, Resistor_SMD:R_0603_1608Metric_Pad0.98x0.95mm_HandSolder, F.Cu at (153.2, 69.9)
- added R22: 0603 0R/1%, Resistor_SMD:R_0603_1608Metric_Pad0.98x0.95mm_HandSolder, F.Cu at (142.6, 51.2)
- added R220: 0603 10K/1%, Resistor_SMD:R_0603_1608Metric_Pad0.98x0.95mm_HandSolder, F.Cu at (153.2, 67.4)
- added R221: 0603 10K/1%, Resistor_SMD:R_0603_1608Metric_Pad0.98x0.95mm_HandSolder, F.Cu at (153.0, 107.1)
- added R222: 0603 10K/1%, Resistor_SMD:R_0603_1608Metric_Pad0.98x0.95mm_HandSolder, F.Cu at (153.0, 104.6)
- added R223: 0603 10K/1%, Resistor_SMD:R_0603_1608Metric_Pad0.98x0.95mm_HandSolder, F.Cu at (153.0, 102.1)
- added R224: 0603 10K/1%, Resistor_SMD:R_0603_1608Metric_Pad0.98x0.95mm_HandSolder, F.Cu at (153.0, 99.6)
- added R225: 0603 10K/1%, Resistor_SMD:R_0603_1608Metric_Pad0.98x0.95mm_HandSolder, F.Cu at (153.0, 97.1)
- added R226: 0603 10K/1%, Resistor_SMD:R_0603_1608Metric_Pad0.98x0.95mm_HandSolder, F.Cu at (153.0, 94.6)
- added R227: 0603 10K/1%, Resistor_SMD:R_0603_1608Metric_Pad0.98x0.95mm_HandSolder, F.Cu at (153.0, 92.1)
- added R23: 0603 0R/1%, Resistor_SMD:R_0603_1608Metric_Pad0.98x0.95mm_HandSolder, F.Cu at (126.2, 49.3)
- added R24: 0603 0R/1%, Resistor_SMD:R_0603_1608Metric_Pad0.98x0.95mm_HandSolder, F.Cu at (108.0, 48.0)
- added R25: 0603 0R/1%, Resistor_SMD:R_0603_1608Metric_Pad0.98x0.95mm_HandSolder, F.Cu at (126.2, 41.3)
- added R26: 0603 0R/1%, Resistor_SMD:R_0603_1608Metric_Pad0.98x0.95mm_HandSolder, F.Cu at (126.2, 43.8)
- added R27: 0603 0R/1%, Resistor_SMD:R_0603_1608Metric_Pad0.98x0.95mm_HandSolder, F.Cu at (126.2, 46.3)
- added R28: 0603 0R/1%, Resistor_SMD:R_0603_1608Metric_Pad0.98x0.95mm_HandSolder, F.Cu at (67.6, 74.4)
- added R29: 0603 0R/1%, Resistor_SMD:R_0603_1608Metric_Pad0.98x0.95mm_HandSolder, F.Cu at (67.6, 77.5)
- added R3: 0603 1K/1%, Resistor_SMD:R_0603_1608Metric_Pad0.98x0.95mm_HandSolder, F.Cu at (80.5, 41.9)
- added R30: 0603 10K/1%, Resistor_SMD:R_0603_1608Metric_Pad0.98x0.95mm_HandSolder, F.Cu at (70.6, 72.5)
- added R31: 0603 12K/1%, Resistor_SMD:R_0603_1608Metric_Pad0.98x0.95mm_HandSolder, F.Cu at (73.3, 66.2)
- added R32: 0603 2K/1%, Resistor_SMD:R_0603_1608Metric_Pad0.98x0.95mm_HandSolder, F.Cu at (69.3, 57.4)
- added R33: 0603 10K/1%, Resistor_SMD:R_0603_1608Metric_Pad0.98x0.95mm_HandSolder, F.Cu at (71.8, 57.4)
- added R34: 0603 10K/1%, Resistor_SMD:R_0603_1608Metric_Pad0.98x0.95mm_HandSolder, F.Cu at (74.3, 57.4)
- added R35: 0603 10K/1%, Resistor_SMD:R_0603_1608Metric_Pad0.98x0.95mm_HandSolder, F.Cu at (76.8, 57.4)
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
Commit message: Updated PCB design
Parts:
- removed R158, R159: 0603 10K/1%, Resistor_SMD:R_0603_1608Metric_Pad0.98x0.95mm_HandSolder
- moved TP27 108.3 mm to (106.2, 122.4), turned to -90 degrees
- moved TP28 107.9 mm to (106.2, 125.4), turned to -90 degrees
- moved LED8 103.2 mm to (150.7, 49.5), turned to -90 degrees
- moved LED7 99.8 mm to (154.2, 49.5), turned to -90 degrees
- moved LED6 96.8 mm to (157.6, 49.5), turned to -90 degrees
- moved R89 96.2 mm to (147.6, 53.5)
- moved TP29 94.2 mm to (194.7, 149.5), turned to 90 degrees
- moved LED5 94.1 mm to (161.0, 49.5), turned to -90 degrees
- moved R88 93.1 mm to (150.7, 53.5)
- moved TP30 91.9 mm to (203.7, 149.4), turned to -90 degrees
- moved R87 90.0 mm to (154.2, 53.6)
- moved R86 87.2 mm to (157.6, 53.6)
- moved TP16 77.7 mm to (100.8, 47.9), turned to 180 degrees
- moved TP22 74.1 mm to (108.3, 41.2), turned to 180 degrees
- moved KEY9 71.6 mm to (95.0, 149.5), turned to -90 degrees
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Connections:
- net /ETH_RXN1 renamed /ETH1_RXN
- net /ETH_RXN2 renamed /ETH2_RXN
- net /ETH_RXP1 renamed /ETH1_RXP
- net /ETH_RXP2 renamed /ETH2_RXP
- net /ETH_TXN1 renamed /ETH1_TXN
- net /ETH_TXN2 renamed /ETH2_TXN
- net /ETH_TXP1 renamed /ETH1_TXP
- net /ETH_TXP2 renamed /ETH2_TXP
- BAT1 pad 2: GND -> VSS
- BTB100x1 pad 190: /EXP_PIN13 -> /BTB_PD3
- BTB100x1 pad 191: /BTB_PD3 -> /EXP_PIN13
- BTB100x1 pad 69: /BTB_PF10 -> unconnected-(BTB100x1-Pad69)
- C100 pad 2: GND -> VSS
- C101 pad 2: GND -> VSS
- C71 pad 1: VSSA -> VSS
- C72 pad 1: VSSA -> VSS
- ESD2 pad 1: Net-(ESD1-A1) -> Net-(ESD2-A1)
- J10 pad 10: /EXP_PIN9 -> /EXP_PIN8
- J10 pad 12: /EXP_PIN10 -> /BTB_PC7
- J10 pad 14: /EXP_PIN11 -> /BTB_PC6
- J10 pad 16: /EXP_PIN12 -> /EXP_PIN7
- J10 pad 2: /BTB_PC6 -> /EXP_PIN12
- J10 pad 4: /BTB_PC7 -> /EXP_PIN11
- J10 pad 6: /EXP_PIN7 -> /EXP_PIN10
- J10 pad 8: /EXP_PIN8 -> /EXP_PIN9
- J7 pad 1: /AKINA_I2C2_SCL -> /AKINA_I2C1_SCL
- J7 pad 13: unconnected-(J7-Pad13) -> /AKINA_I2C2_SCL
- J7 pad 15: unconnected-(J7-Pad15) -> /AKINA_I2C2_SDA
- J7 pad 17: /AKINA_I2C1_SCL -> unconnected-(J7-Pad17)
- J7 pad 19: /AKINA_I2C1_SDA -> unconnected-(J7-Pad19)
- J7 pad 3: /AKINA_I2C2_SDA -> /AKINA_I2C1_SDA
- R29 pad 1: Net-(USB1-A6) -> Net-(ESD2-A1)
- R63 pad 2: /AKINA_BOOT0 -> /AKINA_BOOT1
- R64 pad 2: /AKINA_BOOT1 -> /AKINA_BOOT0
- U12 pad 31: VSSA -> VSS
- U12 pad 33: +3.3VA -> +3V3
- U13 pad 22: /ETH_GPIO0 -> /ETH1_GPIO0
- U13 pad 23: /ETH_GPIO1 -> /ETH1_GPIO1
- U13 pad 24: /ETH_GPIO2 -> /ETH1_GPIO2
- U13 pad 25: /ETH_GPIO3 -> /ETH1_GPIO3
- U13 pad 26: /ETH_RST2 -> /ETH1_RST2
- U13 pad 27: /ETH_SEL -> /ETH1_SEL
- U13 pad 32: /ETH_GPIO4 -> /ETH1_GPIO4
- U13 pad 33: /ETH_GPIO5 -> /ETH1_GPIO5
- U13 pad 34: /ETH_GPIO6 -> /ETH1_GPIO6
- U13 pad 35: /ETH_GPIO7 -> /ETH1_GPIO7
- U14 pad 22: /ETH_GPIO0 -> /ETH2_GPIO0
- U14 pad 23: /ETH_GPIO1 -> /ETH2_GPIO1
- U14 pad 24: /ETH_GPIO2 -> /ETH2_GPIO2
- U14 pad 25: /ETH_GPIO3 -> /ETH2_GPIO3
- U14 pad 26: /ETH_RST2 -> /ETH2_RST2
- U14 pad 27: /ETH_SEL -> /ETH2_SEL
- U14 pad 32: /ETH_GPIO4 -> /ETH2_GPIO4
- U14 pad 33: /ETH_GPIO5 -> /ETH2_GPIO5
- U14 pad 34: /ETH_GPIO6 -> /ETH2_GPIO6
- U14 pad 35: /ETH_GPIO7 -> /ETH2_GPIO7
- USB1 pad 6: Net-(USB1-A6) -> Net-(ESD2-A1)
- USB1 pad 8: Net-(USB1-A6) -> Net-(ESD2-A1)
Routing:
- net VSS: track 0.00 -> 1745.2 mm, vias 0 -> 118
- net +3V3: track 0.00 -> 848.3 mm, vias 0 -> 56
- net +1V8: track 0.00 -> 216.5 mm, vias 0 -> 14
- net /DUT_+3.3V_1: track 0.00 -> 197.6 mm, vias 0 -> 5
- net +5V: track 0.00 -> 178.6 mm, vias 0 -> 1
- net /DUT_VDDA_3.3V_1: track 0.00 -> 168.6 mm, vias 0 -> 2
- net /AKINA_HALL_CH3: track 0.00 -> 151.9 mm, vias 0 -> 4
- net /AKINA_HALL_CH2: track 0.00 -> 143.4 mm, vias 0 -> 4
- net +3.3VA: track 0.00 -> 139.8 mm, vias 0 -> 3
- net /AKINA_USART1_TX: track 0.00 -> 133.5 mm, vias 0 -> 1
- net /AKINA_HALL_CH1: track 0.00 -> 132.3 mm, vias 0 -> 4
- net /AKINA_USART1_RX: track 0.00 -> 129.7 mm, vias 0 -> 1
- net /AKINA_CMP2_IN: track 0.00 -> 110.9 mm, vias 0 -> 2
- net /MC_BKIN_0: track 0.00 -> 107.4 mm
- net /MC_BKIN_1: track 0.00 -> 103.7 mm, vias 0 -> 2
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Other:
- board outline added: 190 x 125 mm
- copper layers 2 -> 4

Commit message: update PCB design
Parts:
- moved J30 83.5 mm to (172.7, 32.4), turned to -90 degrees
- moved J29 65.4 mm to (167.7, 41.6), turned to 90 degrees
- moved BAT1 1.57 mm to (155.0, 39.1)
- moved TP26 0.41 mm to (138.1, 63.0)
- moved R180 0.15 mm to (128.3, 59.0)
- moved R181 0.15 mm to (126.4, 59.0)
- moved R183 0.15 mm to (124.5, 59.0)
- moved R184 0.15 mm to (130.2, 59.0)
- moved R185 0.15 mm to (132.1, 59.0)
- moved R186 0.15 mm to (134.0, 59.0)
- moved R187 0.15 mm to (135.9, 59.0)
Routing:
- net /AKINA_USART3_TX: track 23.7 -> 86.2 mm, vias 1 -> 2
- net /AKINA_USART3_RX: track 25.2 -> 84.0 mm, vias 1 -> 2
- net /AKINA_USART4_TX: track 32.0 -> 85.8 mm
- net /BTB_PD10: track 13.4 -> 66.5 mm, vias 0 -> 1
- net /AKINA_USART4_RX: track 33.3 -> 82.8 mm
- net /BTB_PD9: track 14.2 -> 61.2 mm, vias 0 -> 1
- net /PF10: track 43.9 -> 88.0 mm, vias 1 -> 2
- net /FT_USART2_RX: track 1.85 -> 41.3 mm
- net /PD4: track 26.2 -> 61.2 mm, vias 0 -> 1
- net /PE7: track 10.8 -> 45.2 mm, vias 1 -> 2
- net /FT_USART2_TX: track 2.62 -> 36.1 mm
- net /EXP_PIN7: track 3.36 -> 36.1 mm, vias 1 -> 2
- net /PG4: track 9.12 -> 41.2 mm, vias 1 -> 3
- net /PE8: track 9.11 -> 40.7 mm
- net +3V3: track 848.3 -> 875.9 mm, vias 56 -> 57
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
Commit message: updated PCB design-2023-5-24
Parts:
- moved R203 3.92 mm to (122.3, 125.5), turned to 180 degrees
- moved R40 2.95 mm to (72.3, 115.2)
Connections:
- J4 pad 2: /PG3 -> VSS
Routing:
- net VSS: track 1768.7 -> 1951.0 mm, vias 118 -> 120
- net +3V3: track 875.9 -> 959.1 mm, vias 57 -> 60
- net /FT_USART2_TX: track 36.1 -> 116.6 mm, vias 1 -> 2
- net /FT_USART2_RX: track 41.3 -> 120.9 mm, vias 1 -> 2
- net /STM32_SPI6_NSS: track 8.28 -> 78.2 mm, vias 2 -> 4
- net /STM32_SPI6_SCK: track 6.53 -> 68.6 mm, vias 2 -> 4
- net /STM32_SPI6_MOSI: track 8.14 -> 69.4 mm
- net /PD1: track 10.9 -> 68.7 mm, vias 0 -> 3
- net /PD0: track 12.2 -> 69.6 mm, vias 0 -> 3
- net /PG7: track 15.6 -> 72.7 mm
- net /STM32_SPI6_MISO: track 12.2 -> 63.7 mm
- net /PG6: track 2.54 -> 41.9 mm, vias 0 -> 3
- net /PG5: track 2.54 -> 41.8 mm, vias 0 -> 2
- net /PB0: track 0.00 -> 37.4 mm, vias 0 -> 1
- net /PG1: track 5.76 -> 39.1 mm, vias 0 -> 2
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
Commit message: almost finished the PCB design
Parts:
- removed R205: 0603 10K/1%, Resistor_SMD:R_0603_1608Metric_Pad0.98x0.95mm_HandSolder
- moved R48 1.14 mm to (137.8, 131.1)
- moved R49 1.14 mm to (146.8, 131.1)
- moved R50 1.14 mm to (140.8, 131.1)
- moved R51 1.14 mm to (143.8, 131.1)
- moved TP28 0.77 mm to (105.5, 125.3)
- moved TP27 0.76 mm to (105.5, 122.4)
Connections:
- J5 pad 10: /PB2 -> VSS
- J7 pad 17: unconnected-(J7-Pad17) -> VSS
- J7 pad 19: unconnected-(J7-Pad19) -> VSS
- J8 pad 13: unconnected-(J8-Pad13) -> VSS
- J8 pad 15: unconnected-(J8-Pad15) -> VSS
- J9 pad 10: /BTB_PB2 -> VSS
- R96 pad 1: /STM32_DAC_OUT0 -> /STM32_DAC_OUT1
- R97 pad 1: /STM32_DAC_OUT1 -> /STM32_DAC_OUT2
- U12 pad 48: /PB2 -> /STM32_BOOT1
Routing:
- net /STM32_DAC_OUT2: track 9.33 -> 248.5 mm, vias 1 -> 4
- net /STM32_DAC_OUT1: track 9.96 -> 246.2 mm, vias 1 -> 4
- net VSS: track 1951.0 -> 2138.8 mm, vias 120 -> 122
- net /DUT_VBAT: track 89.3 -> 226.1 mm, vias 4 -> 5
- net /PA0: track 81.9 -> 189.0 mm, vias 3 -> 4
- net /PA1: track 87.6 -> 190.4 mm, vias 4 -> 5
- net /PA2: track 82.2 -> 178.4 mm, vias 3 -> 4
- net /PA3: track 90.8 -> 181.7 mm, vias 3 -> 4
- net /AKINA_I2C1_SDA: track 46.0 -> 128.8 mm
- net /AKINA_I2C1_SCL: track 44.7 -> 120.3 mm
- net /AKINA_SPI1_NSS: track 66.1 -> 140.5 mm
- net /AKINA_I2C2_SDA: track 35.3 -> 108.8 mm, vias 0 -> 2
- net +3V3: track 959.1 -> 1031.5 mm, vias 60 -> 64
- net /AKINA_I2C2_SCL: track 35.8 -> 104.3 mm, vias 0 -> 2
- net /AKINA_ETH_SCK: track 36.3 -> 103.7 mm, vias 1 -> 3
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