File: PSVB_EvalBoard/PSVB_EvalBoard.kicad_pcb (KiCad board)
At the start: 4 copper layers, 190 x 125 mm, 460 parts, among them J10 PIN20, J11 PIN12_2x6, J12 PIN20, J13 PIN6_2x3, J2 PIN2, J29 PIN6_2x3, J3 PIN20, J30 PIN6_2x3, J31 PIN6_2x3, J4 PIN20, J5 PIN20, J6 PIN20, J7 PIN20, J8 PIN20, J9 PIN20, Q1 S9013, U1 SGM2036-ADJ, U11 93LC56BT-IOT, U12 STM32F429ZETx, U13 CH395Q, U14 CH395Q, U15 24LC64ISN, U16 MPU6050, U17 W25Q128JVSIQ, U2 SGM2036-ADJ, U3 SGM2036-ADJ, U4 INA240A1PWR, U5 INA240A1PWR, U6 TM7707, U7 REF3030, U8 REF3025, U9 REF3012, X1 2.4576Mhz, X2 12Mhz_Passive_3225, X3 16Mhz_Passive_3225, X4 30Mhz_3225, X5 30Mhz_3225

Commit message: Finished the PCB layout
Routing:
- net +5V: track 181.9 -> 372.4 mm, vias 1 -> 4
- net /PF8: track 47.9 -> 226.0 mm, vias 1 -> 4
- net /PF7: track 52.8 -> 228.0 mm, vias 1 -> 4
- net /PF4: track 101.9 -> 273.5 mm, vias 4 -> 6
- net /PF3: track 82.1 -> 251.0 mm, vias 5 -> 7
- net /PF6: track 50.4 -> 216.9 mm, vias 1 -> 4
- net /PF1: track 153.8 -> 319.1 mm, vias 3 -> 4
- net /PF0: track 149.4 -> 310.3 mm, vias 1 -> 2
- net /PF5: track 87.5 -> 242.4 mm, vias 3 -> 4
- net /PF10: track 86.9 -> 233.3 mm, vias 2 -> 4
- net /PF13: track 36.3 -> 169.4 mm
- net /PF14: track 35.4 -> 168.4 mm
- net /PF2: track 115.8 -> 247.8 mm, vias 3 -> 4
- net /PF15: track 34.1 -> 165.9 mm
- net /PF11: track 31.6 -> 160.6 mm
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
Commit message: Did some modification.
Routing:
- net /BTB_PF10: track 18.2 -> 57.3 mm, vias 0 -> 1
Changed lines of the file:
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@@
   (segment (start 214.5284 61.00605) (end 214.5284 73.53931) (width 0.1778) (layer "F.Cu") (net 55))
   (segment (start 213.404519 75.325) (end 211.95 75.325) (width 0.1778) (layer "F.Cu") (net 55))
+  (segment (start 215.4936 59.3833) (end 214.341655 59.3833) (width 0.1778) (layer "F.Cu") (net 55))
   (segment (start 215.4936 59.3833) (end 214.993358 59.883542) (width 0.1778) (layer "F.Cu") (net 55))
+  (via (at 214.2236 59.3344) (size 0.8) (drill 0.4) (layers "F.Cu" "B.Cu") (net 55))
   (arc (start 214.993358 59.883542) (mid 214.649239 60.398553) (end 214.5284 61.00605) (width 0.1778) (layer "F.Cu") (net 55))
+  (arc (start 214.341655 59.3833) (mid 214.277764 59.370591) (end 214.2236 59.3344) (width 0.1778) (layer "F.Cu") (net 55))
   (arc (start 214.5284 73.53931) (mid 214.356852 74.401742) (end 213.868306 75.132894) (width 0.1778) (layer "F.Cu") (net 55))
   (arc (start 213.868306 75.132894) (mid 213.655523 75.275073) (end 213.404519 75.325) (width 0.1778) (layer "F.Cu") (net 55))
+  (segment (start 228.2444 89.7636) (end 227.980189 89.499389) (width 0.1778) (layer "In1.Cu") (net 55))
+  (segment (start 215.2396 77.25597) (end 215.2396 75.7428) (width 0.1778) (layer "In1.Cu") (net 55))
+  (segment (start 225.4504 83.8708) (end 223.909588 82.329988) (width 0.1778) (layer "In1.Cu") (net 55))
+  (segment (start 215.2396 75.7428) (end 215.2396 62.79963) (width 0.1778) (layer "In1.Cu") (net 55))
+  (segment (start 218.186 79.9592) (end 218.086514 79.9592) (width 0.1778) (layer "In1.Cu") (net 55))
+  (segment (start 225.789006 84.209406) (end 225.4504 83.8708) (width 0.1778) (layer "In1.Cu") (net 55))
+  (segment (start 214.2236 60.34679) (end 214.2236 59.3344) (width 0.1778) (layer "In1.Cu") (net 55))
+  (segment (start 214.2236 59.3344) (end 214.2236 59.2836) (width 0.1778) (layer "In1.Cu") (net 55))
+  (arc (start 223.909588 82.329988) (mid 221.283583 80.575348) (end 218.186 79.9592) (width 0.1778) (layer "In1.Cu") (net 55))
+  (arc (start 215.2396 62.79963) (mid 215.041563 61.80403) (end 214.4776 60.96) (width 0.1778) (layer "In1.Cu") (net 55))
+  (arc (start 216.0016 79.0956) (mid 215.437638 78.251571) (end 215.2396 77.25597) (width 0.1778) (layer "In1.Cu") (net 55))
+  (arc (start 218.086514 79.9592) (mid 216.958167 79.734758) (end 216.0016 79.0956) (width 0.1778) (layer "In1.Cu") (net 55))
+  (arc (start 226.9744 87.0712) (mid 226.666326 85.522408) (end 225.789006 84.209406) (width 0.1778) (layer "In1.Cu") (net 55))
+  (arc (start 214.4776 60.96) (mid 214.289613 60.678657) (end 214.2236 60.34679) (width 0.1778) (layer "In1.Cu") (net 55))
+  (arc (start 227.980189 89.499389) (mid 227.235796 88.385327) (end 226.9744 87.0712) (width 0.1778) (layer "In1.Cu") (net 55))
   (segment (start 211.95 74.525) (end 211.082946 74.525) (width 0.1778) (layer "F.Cu") (net 56))
   (segment (start 210.01946 75.24706) (end 210.01946 75.316388) (width 0.1778) (layer "F.Cu") (net 56))

Commit message: Fixed some issues.
Connections:
- J24 pad 1: /OPAMP1_IP -> unconnected-(J24-Pad1)
- J24 pad 2: VSS -> unconnected-(J24-Pad2)
- J24 pad 3: /OPAMP1_IN -> unconnected-(J24-Pad3)
- J3 pad 16: /PF9 -> /STM32_USB_ID
- J8 pad 15: VSS -> /BTB_PF9
- U16 pad 25: (no net) -> VSS
Routing:
- net /STM32_USB_ID: track 2.07 -> 57.2 mm, vias 1 -> 3
- net /BTB_PF9: track 18.3 -> 58.9 mm
- net VSS: track 2174.5 -> 2184.5 mm, vias 113 -> 114
- net /TP25: track 19.5 -> 20.8 mm
