File: PSVB_EvalBoard/PSVB_EvalBoard.kicad_sch (KiCad schematic)
At the start: 382 parts, among them J1 PIN2, J1 USB_C_16PIN-Connector, J10 PIN20, J11 PIN20, J12 PIN20, J13 PIN20, J18 Micro_SD_Card, J19 PIN12_2x6, J2 USB_C_16PIN-Connector, J27 PIN6_2x3, J28 PIN20, J6 PIN20, J7 PIN20, J8 PIN20, J9 PIN20, Q1 S9013, U1 STM32F429ZETx, U11 SGM2036-ADJ, U12 TM7707, U13 INA240A2PWR, U14 INA240A2PWR, U15 REF3030, U16 REF3025, U17 REF3012, U2 SGM2036-ADJ, U3 93LC56BT-IOT, U4 SGM2036-ADJ, U5 W25Q128JVSIQ, U6 24LC64ISN, U8 CH395Q, U8 MPU6050, U9 CH395Q, X1 16Mhz_Passive_3225, X2 12Mhz_Passive_3225, X3 30Mhz_3225, X4 30Mhz_3225, X5 2.4576Mhz_Passive_3225

Commit message: update PSVB hardware design
Parts:
- removed C3: 30p, Capacitor_SMD:C_0603_1608Metric_Pad1.08x0.95mm_HandSolder, symbol Device:C
- removed J18: Micro_SD_Card, symbol Connector:Micro_SD_Card
- removed R41: 1K/1%, Resistor_SMD:R_0603_1608Metric_Pad0.98x0.95mm_HandSolder, symbol Device:R
- removed X5: 2.4576Mhz_Passive_3225, Oscillator:Oscillator_SMD_EuroQuartz_XO32-4Pin_3.2x2.5mm_HandSoldering, symbol zgoolib:16Mhz_Passive_3225_4Pin-Oscillator
- added C3: 0603 4.7uF/1%, Capacitor_SMD:C_0603_1608Metric_Pad1.08x0.95mm_HandSolder, symbol Device:C
- added C3: 0603 4.7uF/16V, Capacitor_SMD:C_0603_1608Metric_Pad1.08x0.95mm_HandSolder, symbol Device:C
- added C3: 0603 0.01uF/16V, Capacitor_SMD:C_0603_1608Metric_Pad1.08x0.95mm_HandSolder, symbol Device:C
- added C31: 0.1uF, Capacitor_SMD:C_0603_1608Metric_Pad1.08x0.95mm_HandSolder, symbol Device:C
- added J28: ~, Connector_PinHeader_2.54mm:PinHeader_1x03_P2.54mm_Vertical, symbol zgoolib:PIN3_1x3
- added J29, J30, J31: PIN6_2x3, Connector_PinHeader_2.54mm:PinHeader_2x03_P2.54mm_Vertical, symbol zgoolib:PIN6_2x3
- added R26 (x72): 0603 10K/1%, Resistor_SMD:R_0603_1608Metric_Pad0.98x0.95mm_HandSolder, symbol Device:R
- added R42: 0603 1K/1%, Resistor_SMD:R_0603_1608Metric_Pad0.98x0.95mm_HandSolder, symbol Device:R
- added R55: 0603 100R/1%, Resistor_SMD:R_0603_1608Metric_Pad0.98x0.95mm_HandSolder, symbol Device:R
- added SD1: ~, zgoolib:TF-SMD_TF-02, symbol zgoolib:SD_Socket_SelfLock
- added X1: 2.4576Mhz, Oscillator:Oscillator_SMD_EuroQuartz_XO91-4Pin_7.0x5.0mm_HandSoldering, symbol zgoolib:2.4576Mhz_Sourced_7050_4PIN-Oscillator
- 3V3_LED1: value 3V3_PWR -> 0603 3V3_LED
- 3V3_LED1: value 1V8_PWR -> 0603 1V8_PWR
- 5V_PWR1: value 5V_LED -> 0603 5V_LED
- C1: value 10pF -> 0603 10pF/16V
- C10, C3: value 4.7uF -> 0603 4.7uF/16V
- C16: value 10uF/1% -> 0603 10uF/16V
- C17, C3, C6: value 0.1uF -> 0603 0.1uF/16V
- C18, C19: value 27pF -> 0603 27pF/16V
- C3: value 30p -> 0603 0.1uF/16V
- C3: value 20PF -> 0603 20PF/16V
- C3: value 30p -> 0603 30P/16V
- C3: value 10uF -> 0603 10uF/16V
- C3: value 1uF -> 0603 1uF/16V
- C3: value 1uF -> 0603 0.1uF/16V
- C3: value 1uF -> 0603 4.7uF/16V
- C3: value 3.3uF -> 0603 3.3uF/16V
- C3: value 1uF -> 0603 4.7uF/1%
- C3: value 1uF -> 0603 0.1uF/1%
- F1: value 10V/2A -> 1206 10V/2A
- J2: footprint Connector_USB:USB_C_Receptacle_Palconn_UTC16-G -> zgoolib:USB_C_PIN16
- L2: value 6.8nH/500mA -> 2.2uH/1A; footprint Inductor_SMD:L_0603_1608Metric_Pad1.05x0.95mm_HandSolder -> zgoolib:SWPA3010
- R1, R11, R12, R14, R3, R35, R4, R5, R56, R57, R58, R59, R6: value 10K/1% -> 0603 10K/1%
- R12: value 12K/1% -> 0603 12K/1%
- R13: value 2K/1% -> 0603 2K/1%
- R2: value 1M/1% -> 0603 1M/1%
- R23: value 0603 160K/1% -> 0603 160K/16V
- R23: value 0603 550mR/1% -> 0603 10mR/1%
- R34, R42, R43, R44: value 1K/1% -> 0603 1K/1%
- R8: value 0R/1% -> 0603 0R/1%
- R8: value 0R/1% -> 0603 10K/1%
- U4: renamed from U13; value INA240A2PWR -> INA240A1PWR
- U5: renamed from U14; value INA240A2PWR -> INA240A1PWR
- renumbered JTAG2 to AKINA_JTAG, J26 to J1, J9 to J10, J19 to J11, J28 to J12, J27 to J13, J3 to J14, J5 to J15, J14 to J16, J29 to J17, J22 to J18, J30 to J19, J23 to J20, J4 to J21, J24 to J22, J25 to J23, J15 to J24, J16 to J25, J17 to J26, J21 to J27, J10 to J3, J12 to J4, J11 to J5, J13 to J6, J6 to J7, J7 to J8, J8 to J9, U4 to U1, U3 to U10, U1 to U12, U11 to U3, U12 to U6, U15 to U7, U16 to U8, U17 to U9, X1 to X3, X3 to X4, X4 to X5
Connections:
- net BEEP is gone; now on net STM32_BEEP: R34.1
- net STM32_12BIT_ADC1 is gone; now on net ADC12_IN14: C3.1, R8.2
- net STM32_12BIT_ADC2 is gone; now on net ADC12_IN15: C3.2, R8.2
- net STM32_KEY1 is gone; now on net PA0: KEY1.1
- net STM32_KEY2 is gone; now on net PA1: KEY2.1
- net STM32_KEY3 is gone; now on net PA2: KEY3.1
- net STM32_KEY4 is gone; now on net PA3: KEY4.1
- net VBAT is gone; now on net DUT_VBAT: BAT1.1 (+), C33.1, C34.1
- net VBAT_3.3V is gone; now on net DUT_VBAT: U12.6 (VBAT)
- net VDDA_3.3V is gone; now on net +3.3VA: U12.33 (VDDA)
- net +1V8: no longer C3.2, C3.2, C3.2
- net +3.3VA: now also C3.1, C3.2, C3.2, X1.1 (OE), X1.4 (VDD)
- net +3V3: now also SD1.4 (VDD); no longer R1.2
- net +5V: now also BTB100x1.107, BTB100x1.108
- net AD0: now also U12.109 (PA14)
- net AD3: now also U12.105 (PA13)
- net AD4: now also U12.134 (PB4)
- net AKINA_ETH_SCK: now also BTB100x1.170
- net AKINA_ETH_SCS: now also BTB100x1.169
- net AKINA_ETH_SDI: now also BTB100x1.171
- net AKINA_ETH_SDO: now also BTB100x1.172
- net AKINA_OPA_OUT: now also R55.2
- net DUT_+3.3V_1: now also R1.2
- net PA0: now also U12.34 (PA0), R26.2; no longer R44.1
- net PA1: now also U12.35 (PA1), R26.2; no longer R43.1
- net PA2: now also U12.36 (PA2), R26.2; no longer R42.1
- net PA3: now also U12.37 (PA3), R26.2
- net STM32_DAC_OUT1: now also U12.40 (PA4)
- net STM32_USB_DM: now also U12.75 (PB14)
- net STM32_USB_DP: now also U12.76 (PB15)
- net ST_HALL_CH1: now also U12.60 (PE9)
- net ST_HALL_CH2: now also U12.64 (PE11)
- net ST_HALL_CH3: now also U12.66 (PE13)
- net ST_JTDI: now also U12.110 (PA15)
- net ST_JTDO: now also U12.133 (PB3)
- net TM7707_CS: now also U12.93 (PG8)
- net TM7707_DRDY: now also U12.92 (PG7)
- net TM7707_MISO: now also U12.127 (PG12)
- net TM7707_MOSI: now also U12.129 (PG14)
- net TM7707_SCLK: now also U12.128 (PG13)
- net VSS: now also BTB100x1.109, BTB100x1.110, BTB100x1.111, BTB100x1.164, C3.1, C3.1, C3.2, C31.1, J28.3, SD1.10 (GND), SD1.11 (GND), SD1.12 (GND), SD1.13 (GND), SD1.6 (VSS), X1.2 (GND)
- net PE2: now reaches U12.1 (PE2)
- net PE2: now also R26.1
- net PF0: now reaches U12.10 (PF0)
- net PF0: now also R26.1
- net PA8: now reaches U12.100 (PA8)
- net PA9: now reaches U12.101 (PA9)
- net PA10: now reaches U12.102 (PA10)
- net PA11: now reaches U12.103 (PA11)
- net PA12: now reaches U12.104 (PA12)
- net PF1: now reaches U12.11 (PF1)
- net PF1: now also R26.1
- net SDIO_D2: now reaches U12.111 (PC10)
- net SDIO_D2: now also SD1.1 (DAT2(RSV))
- net SDIO_D3: now reaches U12.112 (PC11)
- net SDIO_D3: now also SD1.2 (CDAT3/CS)
- net SDIO_CK: now reaches U12.113 (PC12)
- net SDIO_CK: now also SD1.5 (CLK)
- net PD0: now reaches U12.114 (PD0)
- net PD0: now also R26.2
- net PD1: now reaches U12.115 (PD1)
- net PD1: now also R26.2
- net SDIO_CMD: now reaches U12.116 (PD2)
- net SDIO_CMD: now also SD1.3 (CMD)
- net SD_CARD_CD: now reaches U12.117 (PD3)
- net SD_CARD_CD: now also SD1.9 (CD)
- net PD4: now reaches U12.118 (PD4)
- net PD4: now also R26.2
- net PD5: now reaches U12.119 (PD5)
- net PD5: now also R26.2
- net PF2: now reaches U12.12 (PF2)
- net PF2: now also R26.1
- net PD6: now reaches U12.122 (PD6)
- net PD6: now also R26.2
- net PD7: now reaches U12.123 (PD7)
- net PD7: now also R26.2
- net PG9: now reaches U12.124 (PG9)
- net PG9: now also R26.2
- net PG10: now reaches U12.125 (PG10)
- net PG10: now also R26.2
- net PG11: now reaches U12.126 (PG11)
- net PG11: now also R26.2
- net PF3: now reaches U12.13 (PF3)
- net PF3: now also R26.1
- net PG15: now reaches U12.132 (PG15)
- net PG15: now also R26.2
- net PB5: now reaches U12.135 (PB5)
- net PB5: now also R26.2
- net PB6: now reaches U12.136 (PB6)
- net PB6: now also R44.1
- net PB7: now reaches U12.137 (PB7)
- net PB7: now also R43.1
- net PB8: now reaches U12.139 (PB8)
- net PB8: now also R42.1
- net PF4: now reaches U12.14 (PF4)
- net PF4: now also R26.1
- net PB9: now reaches U12.140 (PB9)
- net PB9: now also R42.1
- net PE0: now reaches U12.141 (PE0)
- net PE0: now also R26.2
- net PE1: now reaches U12.142 (PE1)
- net PE1: now also R26.2
- net PF5: now reaches U12.15 (PF5)
- net PF5: now also R26.1
- net PF6: now reaches U12.18 (PF6)
- net PF6: now also R26.1
- net PF7: now reaches U12.19 (PF7)
- net PF7: now also R26.1
- net PE3: now reaches U12.2 (PE3)
- net PE3: now also R26.1
- net PF8: now reaches U12.20 (PF8)
- net PF8: now also R26.1
- net PF9: now reaches U12.21 (PF9)
- net PF9: now also R26.1
- net PF10: now reaches U12.22 (PF10)
- net PF10: now also R26.1, R26.2
- net PC0: now reaches U12.26 (PC0)
- net PC0: now also R26.2
- net PC1: now reaches U12.27 (PC1)
- net PC1: now also R26.2
- net PC2: now reaches U12.28 (PC2)
- net PC2: now also R26.2
- net ADC123_IN13: now reaches U12.29 (PC3)
- net ADC123_IN13: now also J28.1
- net PE4: now reaches U12.3 (PE4)
- net PE4: now also R26.1
- net PE5: now reaches U12.4 (PE5)
- net PE5: now also R26.1
- net STM32_DAC_OUT2: now reaches U12.41 (PA5)
- net ADC12_IN14: now reaches U12.44 (PC4)
- net ADC12_IN15: now reaches U12.45 (PC5)
- net PB0: now reaches U12.46 (PB0)
- net PB0: now also R26.2
- net PB1: now reaches U12.47 (PB1)
- net PB1: now also R26.2
- net PB2: now reaches U12.48 (PB2)
- net PB2: now also R26.2
- net PF11: now reaches U12.49 (PF11)
- net PF11: now also R26.2
- net PE6: now reaches U12.5 (PE6)
- net PE6: now also R26.1
- net PF12: now reaches U12.50 (PF12)
- net PF12: now also R26.2
- net PF13: now reaches U12.53 (PF13)
- net PF13: now also R26.2
- net PF14: now reaches U12.54 (PF14)
- net PF14: now also R26.2
- net PF15: now reaches U12.55 (PF15)
- net PF15: now also R26.2
- net PG0: now reaches U12.56 (PG0)
- net PG0: now also R26.2
- net PG1: now reaches U12.57 (PG1)
- net PG1: now also R26.2
- net PE7: now reaches U12.58 (PE7)
- net PE7: now also R26.2
- net PE8: now reaches U12.59 (PE8)
- net PE8: now also R26.2
- net PE10: now reaches U12.63 (PE10)
- net PE10: now also R26.2
- net PE12: now reaches U12.65 (PE12)
- net PE12: now also R26.2
- net PE14: now reaches U12.67 (PE14)
- net PE14: now also R26.2
- net PE15: now reaches U12.68 (PE15)
- net PE15: now also R26.2
- net ST_USART3_TX: now reaches U12.69 (PB10)
- net PC13: now reaches U12.7 (PC13)
- net PC13: now also R26.1
- net ST_USART3_RX: now reaches U12.70 (PB11)
- net STM32_USB_ID: now reaches U12.73 (PB12)
- net STM32_BEEP: now reaches U12.74 (PB13)
- net PD8: now reaches U12.77 (PD8)
- net PD8: now also R26.2
- net PD9: now reaches U12.78 (PD9)
- net PD9: now also R26.2
- net PD10: now reaches U12.79 (PD10)
- net PD10: now also R26.2
- net PC14: now reaches U12.8 (PC14)
- net PC14: now also R26.1
- net PD11: now reaches U12.80 (PD11)
- net PD11: now also R26.2
- net PD12: now reaches U12.81 (PD12)
- net PD12: now also R26.2
- net PD13: now reaches U12.82 (PD13)
- net PD13: now also R26.2
- net PD14: now reaches U12.85 (PD14)
- net PD14: now also R26.2
- net PD15: now reaches U12.86 (PD15)
- net PD15: now also R26.2
- net PG2: now reaches U12.87 (PG2)
- net PG2: now also R26.2
- net PG3: now reaches U12.88 (PG3)
- net PG3: now also R26.2
- net PG4: now reaches U12.89 (PG4)
- net PG4: now also R26.2
- net PC15: now reaches U12.9 (PC15)
- net PC15: now also R26.1
- net PG5: now reaches U12.90 (PG5)
- net PG5: now also R26.2
- net PG6: now reaches U12.91 (PG6)
- net PG6: now also R26.2
- net PC6: now reaches U12.96 (PC6)
- net PC6: now also R26.2
- net PC7: now reaches U12.97 (PC7)
- net PC7: now also R26.2
- net SDIO_D0: now reaches U12.98 (PC8)
- net SDIO_D0: now also SD1.7 (DAT0(D0))
- net SDIO_D1: now reaches U12.99 (PC9)
- net SDIO_D1: now also SD1.8 (DAT1(RSV))
- net BTB_PA0: now reaches BTB100x1.103
- net BTB_PA0: now also R26.1
- net BTB_PA1: now reaches BTB100x1.104
- net BTB_PA1: now also R26.1
- net BTB_PA2: now reaches BTB100x1.105
- net BTB_PA2: now also R26.1
- net BTB_PA3: now reaches BTB100x1.106
- net BTB_PA3: now also R26.1
- net BTB_PG0: now reaches BTB100x1.112
- net BTB_PG0: now also R26.1
- net BTB_PG1: now reaches BTB100x1.113
- net BTB_PG1: now also R26.1
- net BTB_PG2: now reaches BTB100x1.114
- net BTB_PG2: now also R26.1
- net BTB_PG3: now reaches BTB100x1.115
- net BTB_PG3: now also R26.1
- net BTB_PG4: now reaches BTB100x1.116
- net BTB_PG4: now also R26.1
- net BTB_PG5: now reaches BTB100x1.117
- net BTB_PG5: now also R26.1
- net BTB_PG6: now reaches BTB100x1.118
- net BTB_PG6: now also R26.1
- net BTB_PE7: now reaches BTB100x1.119
- net BTB_PE7: now also R26.1
- net BTB_PE8: now reaches BTB100x1.120
- net BTB_PE8: now also R26.1
- net BTB_PE10: now reaches BTB100x1.121
- net BTB_PE10: now also R26.1
- net BTB_PE12: now reaches BTB100x1.122
- net BTB_PE12: now also R26.1
- net BTB_PE14: now reaches BTB100x1.123
- net BTB_PE14: now also R26.1
- net BTB_PE15: now reaches BTB100x1.124
- net BTB_PE15: now also R26.1
- net BTB_PE0: now reaches BTB100x1.125
- net BTB_PE0: now also R26.1
- net BTB_PE1: now reaches BTB100x1.126
- net BTB_PE1: now also R26.1
- net BTB_PG15: now reaches BTB100x1.127
- net BTB_PG15: now also R26.1
- net BTB_PB5: now reaches BTB100x1.128
- net BTB_PB5: now also R26.1
- net EXP_PIN3: now reaches BTB100x1.129
- net EXP_PIN4: now reaches BTB100x1.130
- net EXP_PIN5: now reaches BTB100x1.131
- net EXP_PIN6: now reaches BTB100x1.132
- net AKINA_USART1_TX: now reaches BTB100x1.15
- net AKINA_USART1_TX: now also J29.1
- net AKINA_USART1_RX: now reaches BTB100x1.16
- net AKINA_USART1_RX: now also J29.2
- net BTB_PG9: now reaches BTB100x1.160
- net BTB_PG9: now also R26.1
- net BTB_PG10: now reaches BTB100x1.161
- net BTB_PG10: now also R26.1
- net BTB_PG11: now reaches BTB100x1.162
- net BTB_PG11: now also R26.1
- net DUT_VBAT: now reaches BTB100x1.163
- net BTB_PB0: now reaches BTB100x1.165
- net BTB_PB0: now also R26.1
- net BTB_PB1: now reaches BTB100x1.166
- net BTB_PB1: now also R26.1
- net BTB_PB2: now reaches BTB100x1.167
- net BTB_PB2: now also R26.1
- net EXP_PIN7: now reaches BTB100x1.168
- net BTB_PC6: now reaches BTB100x1.173
- net BTB_PC6: now also R26.1
- net BTB_PC7: now reaches BTB100x1.174
- net BTB_PC7: now also R26.1
- net EXP_PIN8: now reaches BTB100x1.175
- net EXP_PIN9: now reaches BTB100x1.176
- net EXP_PIN10: now reaches BTB100x1.177
- net EXP_PIN11: now reaches BTB100x1.178
- net EXP_PIN12: now reaches BTB100x1.179
- net BTB_PD8: now reaches BTB100x1.180
- net BTB_PD8: now also R26.1
- net BTB_PD9: now reaches BTB100x1.181
- net BTB_PD9: now also R26.1
- net BTB_PD10: now reaches BTB100x1.182
- net BTB_PD10: now also R26.1
- net BTB_PD11: now reaches BTB100x1.183
- net BTB_PD11: now also R26.1
- net BTB_PD12: now reaches BTB100x1.184
- net BTB_PD12: now also R26.1
- net BTB_PD13: now reaches BTB100x1.185
- net BTB_PD13: now also R26.1
- net BTB_PD14: now reaches BTB100x1.186
- net BTB_PD14: now also R26.1
- net BTB_PD15: now reaches BTB100x1.187
- net BTB_PD15: now also R26.1
- net BTB_PD0: now reaches BTB100x1.188
- net BTB_PD0: now also R26.1
- net BTB_PD1: now reaches BTB100x1.189
- net BTB_PD1: now also R26.1
- net EXP_PIN13: now reaches BTB100x1.190
- net BTB_PD3: now reaches BTB100x1.191
- net BTB_PD3: now also R26.1
- net BTB_PD4: now reaches BTB100x1.192
- net BTB_PD4: now also R26.1
- net BTB_PD5: now reaches BTB100x1.193
- net BTB_PD5: now also R26.1
- net BTB_PD6: now reaches BTB100x1.194
- net BTB_PD6: now also R26.1
- net BTB_PD7: now reaches BTB100x1.195
- net BTB_PD7: now also R26.1
- net AKINA_USART2_TX: now reaches BTB100x1.196
- net AKINA_USART2_TX: now also J29.5
- net AKINA_USART2_RX: now reaches BTB100x1.197
- net AKINA_USART2_RX: now also J29.6
- net BTB_PF0: now reaches BTB100x1.31
- net BTB_PF0: now also R26.2
- net BTB_PF1: now reaches BTB100x1.32
- net BTB_PF1: now also R26.2
- net BTB_PF2: now reaches BTB100x1.33
- net BTB_PF2: now also R26.2
- net BTB_PF3: now reaches BTB100x1.34
- net BTB_PF3: now also R26.2
- net BTB_PF4: now reaches BTB100x1.35
- net BTB_PF4: now also R26.2
- net BTB_PF5: now reaches BTB100x1.36
- net BTB_PF5: now also R26.2
- net BTB_PF6: now reaches BTB100x1.37
- net BTB_PF6: now also R26.2
- net BTB_PF7: now reaches BTB100x1.38
- net BTB_PF7: now also R26.2
- net BTB_PF8: now reaches BTB100x1.39
- net BTB_PF8: now also R26.2
- net BTB_PF9: now reaches BTB100x1.40
- net BTB_PF9: now also R26.2
- net BTB_PF10: now reaches BTB100x1.41
- net BTB_PF10: now also BTB100x1.69, R26.1, R26.2
- net BTB_PE2: now reaches BTB100x1.51
- net BTB_PE2: now also R26.2
- net BTB_PE3: now reaches BTB100x1.52
- net BTB_PE3: now also R26.2
- net BTB_PE4: now reaches BTB100x1.53
- net BTB_PE4: now also R26.2
- net BTB_PE5: now reaches BTB100x1.54
- net BTB_PE5: now also R26.2
- net BTB_PE6: now reaches BTB100x1.55
- net BTB_PE6: now also R26.2
- net BTB_PC0: now reaches BTB100x1.60
- net BTB_PC0: now also R26.1
- net BTB_PC1: now reaches BTB100x1.61
- net BTB_PC1: now also R26.1
- net BTB_PC2: now reaches BTB100x1.62
- net BTB_PC2: now also R26.1
- net EXP_PIN1: now reaches BTB100x1.63
- net BTB_PC13: now reaches BTB100x1.64
- net BTB_PC13: now also R26.2
- net BTB_PC14: now reaches BTB100x1.65
- net BTB_PC14: now also R26.2
- net BTB_PC15: now reaches BTB100x1.66
- net BTB_PC15: now also R26.2
- net AKINA_USART3_TX: now reaches BTB100x1.67
- net AKINA_USART3_TX: now also J30.1, J31.1
- net AKINA_USART3_RX: now reaches BTB100x1.68
- net AKINA_USART3_RX: now also J30.2, J31.2
- net BTB_PF11: now reaches BTB100x1.70
- net BTB_PF11: now also R26.1
- net BTB_PF12: now reaches BTB100x1.71
- net BTB_PF12: now also R26.1
- net BTB_PF13: now reaches BTB100x1.72
- net BTB_PF13: now also R26.1
- net BTB_PF14: now reaches BTB100x1.73
- net BTB_PF14: now also R26.1
- net BTB_PF15: now reaches BTB100x1.74
- net BTB_PF15: now also R26.1
- net AKINA_USART4_TX: now reaches BTB100x1.77
- net AKINA_USART4_TX: now also J30.5, J31.5
- net AKINA_USART4_RX: now reaches BTB100x1.78
- net AKINA_USART4_RX: now also J30.6, J31.6
- net EXP_PIN2: now reaches BTB100x1.79
- net at U6.2 (MCLK_IN): now also X1.3 (OUT)
- net VCORE: now reaches C3.2, U10.12 (VCORE), U10.37 (VCORE), U10.49 (VREGOUT), U10.64 (VCORE)
- net VCORE: now also C3.2, C3.2, C3.2
- net at LED4.2 (A): now also R42.2
- net AKINA_ETH_RXD renamed ETH1_RXD
- net AKINA_ETH_TXD renamed ETH1_TXD
- net STM32_ETH_RXD renamed ETH2_RXD
- net STM32_ETH_TXD renamed ETH2_TXD
- new net: C31.2, J28.2, R55.1
- new net FT_USART1_RX: J29.3, J30.3
- new net FT_USART1_TX: J29.4, J30.4
- new net FT_USART2_RX: J31.3
- new net FT_USART2_TX: J31.4
- new net PD3: R26.2
- no-connect marks 1 -> 0
Other:
- note added: "20V/V"
- note added: "AKINA Single Ended OPAMP Output"
- note added: "AKINA USART Selection"
- note added: "BTB Board PIN"
- note added: "CH395Q USART Selection"
- note added: "Ethernet SPI"
- note added: "RTC VBAT"
- note added: "USART1"
- note added: "USART2"
- note added: "USART3"
- note added: "USART4"
- note added: "base"
- note added: "collector"
- note added: "donot solder"
- note added: "emitter"
- moved on the sheet: 3V3_LED1, BEEP1, BTB100x1, C1, C3, D1, Q1, R1, R22, R23, R34, R8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

Commit message: Almost finished the schematic design
Parts:
- R32: value 10K/1% -> 0603 10K/1%
Connections:
- net FT_USART1_RX is gone; now on net FT_USART2_RX: J29.3, J30.3
- net FT_USART1_TX is gone; now on net FT_USART2_TX: J29.4, J30.4
- net SDIO_CK is gone; now on net PC12: SD1.5 (CLK), U12.113 (PC12)
- net SDIO_CMD is gone; now on net PD2: SD1.3 (CMD), U12.116 (PD2)
- net SDIO_D0 is gone; now on net PC8: SD1.7 (DAT0(D0)), U12.98 (PC8)
- net SDIO_D1 is gone; now on net PC9: SD1.8 (DAT1(RSV)), U12.99 (PC9)
- net SDIO_D2 is gone; now on net PC10: SD1.1 (DAT2(RSV)), U12.111 (PC10)
- net SDIO_D3 is gone; now on net PC11: SD1.2 (CDAT3/CS), U12.112 (PC11)
- net SD_CARD_CD is gone; now on net PD3: SD1.9 (CD), U12.117 (PD3)
- net ST_USART3_RX is gone; now on net FT_USART3_TX: U12.70 (PB11)
- net ST_USART3_TX is gone; now on net FT_USART3_RX: U12.69 (PB10)
- net TM7707_CS is gone; now on net STM32_SPI6_NSS: U12.93 (PG8), U6.4 (~{CS})
- net TM7707_DRDY is gone; now on net PG7: U12.92 (PG7), U6.12 (~{DRDY})
- net TP1 is gone; now on net +3.3VA: TP1.1
- net TP10 is gone; now on net +3V3: TP10.1
- net TP11 is gone; now on net VSS: TP11.1
- net TP12 is gone; now on net +1V8: TP12.1
- net TP13 is gone; now on net VSS: TP13.1
- net TP14 is gone; now on net AIN1+: TP14.1
- net TP15 is gone; now on net AIN1-: TP15.1
- net TP2 is gone; now on net VSS: TP2.1
- net TP22 is gone; now on net AIN2+: TP22.1
- net TP23 is gone; now on net AIN2-: TP23.1
- net TP26 is gone; now on net VSS: TP26.1
- net TP28 is gone; now on net VSS: TP28.1
- net TP29 is gone; now on net AKINA_RESET: TP29.1
- net TP30 is gone; now on net VSS: TP30.1
- net TP4 is gone; now on net AIN2-: TP4.1
- net TP5 is gone; now on net VSS: TP5.1
- net TP6 is gone; now on net ADC12_IN15: TP6.1
- net TP7 is gone; now on net INA240_Output1: TP7.1
- net TP8 is gone; now on net VSS: TP8.1
- net TP9 is gone; now on net ADC12_IN14: TP9.1
- net +3V3: now also J5.2, J5.4, J6.18, J6.20
- net AKINA_BLK: now also J7.6
- net AKINA_D_C: now also J7.4
- net AKINA_ETH_SCK: now also J9.16
- net AKINA_ETH_SCS: now also J9.14
- net AKINA_ETH_SDI: now also J9.18
- net AKINA_ETH_SDO: now also J9.20
- net AKINA_I2C1_SCL: now also J7.17
- net AKINA_I2C1_SDA: now also J7.19
- net AKINA_I2C2_SCL: now also J7.1
- net AKINA_I2C2_SDA: now also J7.3
- net AKINA_KEY1: now also J8.12
- net AKINA_KEY2: now also J8.14
- net AKINA_KEY3: now also J8.16
- net AKINA_KEY4: now also J8.18
- net AKINA_LED0: now also J7.14
- net AKINA_LED1: now also J7.16
- net AKINA_LED2: now also J7.18
- net AKINA_LED3: now also J7.20
- net AKINA_SCREEN_RST: now also J7.2
- net AKINA_SPI1_MISO: now also J7.7
- net AKINA_SPI1_MOSI: now also J7.9
- net AKINA_SPI1_NSS: now also J7.11
- net AKINA_SPI1_SCK: now also J7.5
- net AKINA_SPI2_MOSI: now also J7.10
- net AKINA_SPI2_NSS: now also J7.12
- net AKINA_SPI2_SCK: now also J7.8
- net AKINA_USART3_RX: no longer J31.2
- net AKINA_USART3_TX: no longer J31.1
- net AKINA_USART4_RX: no longer J31.6
- net AKINA_USART4_TX: no longer J31.5
- net BTB_PB0: now also J9.6
- net BTB_PB1: now also J9.8
- net BTB_PB2: now also J9.10
- net BTB_PC0: now also J8.20
- net BTB_PC1: now also J8.1
- net BTB_PC13: now also J8.7
- net BTB_PC14: now also J8.9
- net BTB_PC15: now also J8.11
- net BTB_PC2: now also J8.3
- net BTB_PC6: now also J10.2
- net BTB_PC7: now also J10.4
- net BTB_PD0: now also J10.17
- net BTB_PD1: now also J10.19
- net BTB_PD10: now also J10.5
- net BTB_PD11: now also J10.7
- net BTB_PD12: now also J10.9
- net BTB_PD13: now also J10.11
- net BTB_PD14: now also J10.13
- net BTB_PD15: now also J10.15
- net BTB_PD3: now also J10.20
- net BTB_PD8: now also J10.1
- net BTB_PD9: now also J10.3
- net BTB_PE2: now also J8.2
- net BTB_PE3: now also J8.4
- net BTB_PE4: now also J8.6
- net BTB_PE5: now also J8.8
- net BTB_PE6: now also J8.10
- net BTB_PE7: now also J9.9
- net BTB_PE8: now also J9.11
- net BTB_PF10: now also J8.17
- net BTB_PG0: now also J9.1
- net BTB_PG1: now also J9.2
- net BTB_PG2: now also J9.4
- net BTB_PG3: now also J9.3
- net BTB_PG4: now also J9.5
- net BTB_PG5: now also J9.7
- net BTB_PG6: now also J9.12
- net ETH1_RXD: now also J31.2
- net ETH1_TXD: now also J31.1
- net ETH2_RXD: now also J31.6
- net ETH2_TXD: now also J31.5
- net EXP_PIN1: now also J8.5
- net EXP_PIN10: now also J10.12
- net EXP_PIN11: now also J10.14
- net EXP_PIN12: now also J10.16
- net EXP_PIN13: now also J10.18
- net EXP_PIN2: now also J8.19
- net EXP_PIN3: now also J9.13
- net EXP_PIN4: now also J9.15
- net EXP_PIN5: now also J9.17
- net EXP_PIN6: now also J9.19
- net EXP_PIN7: now also J10.6
- net EXP_PIN8: now also J10.8
- net EXP_PIN9: now also J10.10
- net FT_USART2_RX: now also U10.27 (BDBUS1); no longer J31.3
- net FT_USART2_TX: now also U10.26 (BDBUS0); no longer J31.4
- net FT_USART3_RX: now also U10.39 (CDBUS1)
- net FT_USART3_TX: now also U10.38 (CDBUS0)
- net PA0: now also J5.7
- net PA1: now also J5.9
- net PA10: now also J6.9
- net PA11: now also J6.11
- net PA12: now also J6.13
- net PA2: now also J5.11
- net PA3: now also J5.13
- net PA8: now also J6.5
- net PA9: now also J6.7
- net PB0: now also J5.6
- net PB1: now also J5.8
- net PB2: now also J5.10
- net PC0: now also J5.1
- net PC1: now also J5.3
- net PC13: now also J3.11
- net PC14: now also J3.13
- net PC15: now also J3.15
- net PC2: now also J5.5
- net PC6: now also J4.14
- net PC7: now also J4.16
- net PD0: now also J6.2
- net PD1: now also J6.4
- net PD10: now also J4.5
- net PD11: now also J4.7
- net PD12: now also J4.9
- net PD13: now also J4.11
- net PD14: now also J4.13
- net PD15: now also J4.15
- net PD3: now also J6.8
- net PD4: now also J6.10
- net PD5: now also J6.12
- net PD6: now also J6.14
- net PD7: now also J6.16
- net PD8: now also J4.1
- net PD9: now also J4.3
- net PE2: now also J3.1
- net PE3: now also J3.3
- net PE4: now also J3.5
- net PE5: now also J3.7
- net PE6: now also J3.9
- net PE7: now also J5.16
- net PE8: now also J5.18
- net PF0: now also J3.17
- net PF1: now also J3.19
- net PF10: now also J3.18
- net PF2: now also J3.2
- net PF3: now also J3.4
- net PF4: now also J3.6
- net PF5: now also J3.8
- net PF6: now also J3.10; no longer U12.18 (PF6)
- net PF7: now also J3.12; no longer U12.19 (PF7)
- net PF8: now also J3.14; no longer U12.20 (PF8)
- net PF9: now also J3.16; no longer U12.21 (PF9)
- net PG0: now also J5.12
- net PG1: now also J5.14
- net PG2: now also J4.17
- net PG3: now also J4.19, J4.2
- net PG4: now also J4.4
- net PG5: now also J4.6
- net PG6: now also J4.8
- net STM32_ETH_SCK: now also U12.19 (PF7)
- net STM32_ETH_SCS: now also U12.18 (PF6)
- net STM32_ETH_SDI: now also U12.20 (PF8)
- net STM32_ETH_SDO: now also U12.21 (PF9)
- net TP24: now also C31.2, J13.2, R55.2
- net TP25: now also C31.2, J13.4, R55.2
- net TP27: now also C31.2, J28.2, R55.1
- net TP3: now also L2.1, R23.2, U3.5 (VOUT)
- net VSS: now also J3.20, J4.18, J4.20, J5.19, J5.20
- net PA6: now reaches U12.42 (PA6)
- net PA6: now also J5.15
- net PA7: now reaches U12.43 (PA7)
- net PA7: now also J5.17
- net PC8: now reaches J6.1
- net PC10: now reaches J6.15
- net PC11: now reaches J6.17
- net PC12: now reaches J6.19
- net PC9: now reaches J6.3
- net PD2: now reaches J6.6
- net FT_USART4_TX: now reaches U10.48 (DDBUS0)
- net FT_USART4_TX: now also J31.4
- net FT_USART4_RX: now reaches U10.52 (DDBUS1)
- net FT_USART4_RX: now also J31.3
- net PG7: now reaches J4.10
- net STM32_SPI6_NSS: now reaches J4.12
- net TM7707_MISO renamed STM32_SPI6_MISO
- net TM7707_MOSI renamed STM32_SPI6_MOSI
- net TM7707_SCLK renamed STM32_SPI6_SCK
Other:
- moved on the sheet: BAT1, C33, C34, R32

Commit message: update PCB design
Parts:
- BAT1: footprint PUTUO-MCU:CR1220_Holder -> zgoolib:CR1220_Holder
- KEY5: footprint PUTUO-MCU:5Axises_Key -> zgoolib:5Axises_Key
- R23: footprint Resistor_SMD:R_0603_1608Metric_Pad0.98x0.95mm_HandSolder -> Resistor_SMD:R_1206_3216Metric_Pad1.30x1.75mm_HandSolder
- renumbered AKINA_JTAG to AKINA_JTAG1, U8 to U13, U9 to U14, J1 to USB1, J2 to USB2
Changed lines of the file:
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@@
       (project "PSVB_EvalBoard"
         (path "/f2b0a56f-d786-40ff-9774-78e3f95871c8"
-          (reference "ST_RESET") (unit 1)
+          (reference "ST_RESET1") (unit 1)
         )
       )
@@
   (symbol (lib_id "zgoolib:USB_C_16PIN-Connector") (at 81.28 618.49 0) (mirror x) (unit 1)
     (in_bom yes) (on_board yes) (dnp no)
-    (property "Reference" "J2" (at 80.645 640.08 0)
+    (property "Reference" "USB2" (at 80.645 640.08 0)
       (effects (font (size 1.27 1.27)))
     )
@@
       (project "PSVB_EvalBoard"
         (path "/f2b0a56f-d786-40ff-9774-78e3f95871c8"
-          (reference "J2") (unit 1)
+          (reference "USB2") (unit 1)
         )
       )
@@
       (project "PSVB_EvalBoard"
         (path "/f2b0a56f-d786-40ff-9774-78e3f95871c8"
-          (reference "C86") (unit 1)
+          (reference "C97") (unit 1)
         )
       )
@@
       (project "PSVB_EvalBoard"
         (path "/f2b0a56f-d786-40ff-9774-78e3f95871c8"
-          (reference "3V3_PWR") (unit 1)
+          (reference "3V3_PWR1") (unit 1)
         )
       )
@@
       (effects (font (size 1.27 1.27)))
     )
-    (property "Footprint" "PUTUO-MCU:CR1220_Holder" (at 845.82 128.27 0)
+    (property "Footprint" "zgoolib:CR1220_Holder" (at 845.82 128.27 0)
       (effects (font (size 1.27 1.27)) hide)
     )
@@
   (symbol (lib_id "Device:C") (at 811.911 133.477 0) (unit 1)
     (in_bom yes) (on_board yes) (dnp no)
-    (property "Reference" "C33" (at 807.847 129.413 0)
+    (property "Reference" "C33" (at 806.45 129.54 0)
       (effects (font (size 1.27 1.27)) (justify left))
     )
@@
       (project "PSVB_EvalBoard"
         (path "/f2b0a56f-d786-40ff-9774-78e3f95871c8"
-          (reference "C97") (unit 1)
+          (reference "C100") (unit 1)
         )
       )
@@
   (symbol (lib_id "zgoolib:USB_C_16PIN-Connector") (at 303.53 71.12 0) (mirror x) (unit 1)
     (in_bom yes) (on_board yes) (dnp no)
-    (property "Reference" "J1" (at 293.37 52.07 0)
+    (property "Reference" "USB1" (at 295.91 52.07 0)
       (effects (font (size 1.27 1.27)))
     )
@@
       (project "PSVB_EvalBoard"
         (path "/f2b0a56f-d786-40ff-9774-78e3f95871c8"
-          (reference "J1") (unit 1)
+          (reference "USB1") (unit 1)
         )
       )
@@
       (effects (font (size 1.27 1.27)))
     )
-    (property "Footprint" "PUTUO-MCU:5Axises_Key" (at 863.6 457.2 0)
+    (property "Footprint" "zgoolib:5Axises_Key" (at 863.6 457.2 0)
       (effects (font (size 1.27 1.27)) hide)
     )
@@
       (project "PSVB_EvalBoard"
         (path "/f2b0a56f-d786-40ff-9774-78e3f95871c8"
-          (reference "5V_PWR") (unit 1)
+          (reference "5V_PWR1") (unit 1)
         )
       )
@@
       (project "PSVB_EvalBoard"
         (path "/f2b0a56f-d786-40ff-9774-78e3f95871c8"
-          (reference "U6") (unit 1)
+          (reference "U16") (unit 1)
         )
       )
@@
       (project "PSVB_EvalBoard"
         (path "/f2b0a56f-d786-40ff-9774-78e3f95871c8"
-          (reference "1V8_PWR") (unit 1)
+          (reference "1V8_PWR1") (unit 1)
         )
       )
@@
       (effects (font (size 1.27 1.27)) (justify left))
     )
-    (property "Footprint" "Resistor_SMD:R_0603_1608Metric_Pad0.98x0.95mm_HandSolder" (at 33.782 318.77 90)
+    (property "Footprint" "Resistor_SMD:R_1206_3216Metric_Pad1.30x1.75mm_HandSolder" (at 33.782 318.77 90)
       (effects (font (size 1.27 1.27)) hide)
     )
@@
       (project "PSVB_EvalBoard"
         (path "/f2b0a56f-d786-40ff-9774-78e3f95871c8"
-          (reference "U5") (unit 1)
+          (reference "U15") (unit 1)
         )
       )
@@
   (symbol (lib_id "Device:C") (at 825.627 133.35 0) (unit 1)
     (in_bom yes) (on_board yes) (dnp no)
-    (property "Reference" "C34" (at 821.563 129.286 0)
+    (property "Reference" "C34" (at 820.42 129.54 0)
       (effects (font (size 1.27 1.27)) (justify left))
     )
@@
       (project "PSVB_EvalBoard"
         (path "/f2b0a56f-d786-40ff-9774-78e3f95871c8"
-          (reference "C98") (unit 1)
+          (reference "C101") (unit 1)
         )
       )
@@
       (project "PSVB_EvalBoard"
         (path "/f2b0a56f-d786-40ff-9774-78e3f95871c8"
-          (reference "C93") (unit 1)
+          (reference "C99") (unit 1)
         )
       )
@@
       (effects (font (size 1.27 1.27)) (justify left))
     )
-    (property "Footprint" "Resistor_SMD:R_0603_1608Metric_Pad0.98x0.95mm_HandSolder" (at 33.782 242.57 90)
+    (property "Footprint" "Resistor_SMD:R_1206_3216Metric_Pad1.30x1.75mm_HandSolder" (at 33.782 242.57 90)
       (effects (font (size 1.27 1.27)) hide)
     )
@@
   (symbol (lib_id "zgoolib:PIN10_2x5") (at 374.65 242.57 0) (unit 1)
     (in_bom yes) (on_board yes) (dnp no)
-    (property "Reference" "AKINA_JTAG" (at 374.65 251.46 0)
+    (property "Reference" "AKINA_JTAG1" (at 374.65 251.46 0)
       (effects (font (size 1.27 1.27)))
     )
@@
       (project "PSVB_EvalBoard"
         (path "/f2b0a56f-d786-40ff-9774-78e3f95871c8"
-          (reference "AKINA_JTAG") (unit 1)
+          (reference "AKINA_JTAG1") (unit 1)
         )
       )
@@
   (symbol (lib_id "zgoolib:CH395Q") (at 671.83 81.28 0) (unit 1)
     (in_bom yes) (on_board yes) (dnp no)
-    (property "Reference" "U8" (at 646.43 52.07 0)
+    (property "Reference" "U13" (at 646.43 52.07 0)
       (effects (font (size 1.27 1.27)))
     )
@@
       (project "PSVB_EvalBoard"
         (path "/f2b0a56f-d786-40ff-9774-78e3f95871c8"
-          (reference "U8") (unit 1)
+          (reference "U13") (unit 1)
         )
       )
@@
       (project "PSVB_EvalBoard"
         (path "/f2b0a56f-d786-40ff-9774-78e3f95871c8"
-          (reference "U7") (unit 1)
+          (reference "U17") (unit 1)
         )
       )
@@
       (project "PSVB_EvalBoard"
         (path "/f2b0a56f-d786-40ff-9774-78e3f95871c8"
-          (reference "ST_JTAG") (unit 1)
+          (reference "ST_JTAG1") (unit 1)
         )
       )
@@
       (project "PSVB_EvalBoard"
         (path "/f2b0a56f-d786-40ff-9774-78e3f95871c8"
-          (reference "AKINA_RESET") (unit 1)
+          (reference "AKINA_RESET1") (unit 1)
         )
       )
@@
       (project "PSVB_EvalBoard"
         (path "/f2b0a56f-d786-40ff-9774-78e3f95871c8"
-          (reference "C87") (unit 1)
+          (reference "C98") (unit 1)
         )
       )
@@
   (symbol (lib_id "zgoolib:CH395Q") (at 673.1 198.12 0) (unit 1)
     (in_bom yes) (on_board yes) (dnp no)
-    (property "Reference" "U9" (at 647.7 168.91 0)
+    (property "Reference" "U14" (at 647.7 168.91 0)
       (effects (font (size 1.27 1.27)))
     )
@@
       (project "PSVB_EvalBoard"
         (path "/f2b0a56f-d786-40ff-9774-78e3f95871c8"
-          (reference "U9") (unit 1)
+          (reference "U14") (unit 1)
         )
       )

Commit message: Updated PCB design
Parts:
- removed R26 (x2): 0603 10K/1%, Resistor_SMD:R_0603_1608Metric_Pad0.98x0.95mm_HandSolder, symbol Device:R
- removed T10, T5, T6, T7, T8, T9: ~, zgoolib:M3_Whole, symbol zgoolib:M3_Whole
Connections:
- net GND is gone; now on net VSS: BAT1.2 (-), C33.2, C34.2
- net VSSA is gone; now on net VSS: C3.1, C3.1, U12.31 (VSSA)
- net +3.3VA: no longer U12.33 (VDDA)
- net +3V3: now also U12.33 (VDDA)
- net AKINA_BOOT0: now also R6.2; no longer R5.2
- net AKINA_BOOT1: now also R5.2; no longer R6.2
- net AKINA_I2C1_SCL: now also J7.1; no longer J7.17
- net AKINA_I2C1_SDA: now also J7.3; no longer J7.19
- net AKINA_I2C2_SCL: now also J7.13; no longer J7.1
- net AKINA_I2C2_SDA: now also J7.15; no longer J7.3
- net BTB_PC6: now also J10.14; no longer J10.2
- net BTB_PC7: now also J10.12; no longer J10.4
- net BTB_PD3: now also BTB100x1.190; no longer BTB100x1.191
- net BTB_PF10: no longer BTB100x1.69
- net EXP_PIN10: now also J10.6; no longer J10.12
- net EXP_PIN11: now also J10.4; no longer J10.14
- net EXP_PIN12: now also J10.2; no longer J10.16
- net EXP_PIN13: now also BTB100x1.191; no longer BTB100x1.190
- net EXP_PIN7: now also J10.16; no longer J10.6
- net EXP_PIN8: now also J10.10; no longer J10.8
- net EXP_PIN9: now also J10.8; no longer J10.10
- net at ESD1.1 (A1), R8.1, USB1.5 (B7)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: no longer ESD1.1 (A1)
- net at R8.1, USB1.6 (A6), USB1.8 (B6): now also ESD1.1 (A1)
- net ETH_GPIO0 renamed ETH1_GPIO0
- net ETH1_GPIO0: no longer U14.22 (GPIO0)
- net ETH_GPIO1 renamed ETH1_GPIO1
- net ETH1_GPIO1: no longer U14.23 (GPIO1)
- net ETH_GPIO2 renamed ETH1_GPIO2
- net ETH1_GPIO2: no longer U14.24 (GPIO2)
- net ETH_GPIO3 renamed ETH1_GPIO3
- net ETH1_GPIO3: no longer U14.25 (RDY/GPIO3)
- net ETH_GPIO4 renamed ETH1_GPIO4
- net ETH1_GPIO4: no longer U14.32 (GPIO4)
- net ETH_GPIO5 renamed ETH1_GPIO5
- net ETH1_GPIO5: no longer U14.33 (GPIO5)
- net ETH_GPIO6 renamed ETH1_GPIO6
- net ETH1_GPIO6: no longer U14.34 (GPIO6)
- net ETH_GPIO7 renamed ETH1_GPIO7
- net ETH1_GPIO7: no longer U14.35 (GPIO7)
- net ETH_RST2 renamed ETH1_RST2
- net ETH1_RST2: no longer U14.26 (RST)
- net ETH_RXN1 renamed ETH1_RXN
- net ETH_RXN2 renamed ETH2_RXN
- net ETH_RXP1 renamed ETH1_RXP
- net ETH_RXP2 renamed ETH2_RXP
- net ETH_SEL renamed ETH1_SEL
- net ETH1_SEL: no longer U14.27 (SEL)
- net ETH_TXN1 renamed ETH1_TXN
- net ETH_TXN2 renamed ETH2_TXN
- net ETH_TXP1 renamed ETH1_TXP
- net ETH_TXP2 renamed ETH2_TXP
- new net ETH2_GPIO0: U14.22 (GPIO0)
- new net ETH2_GPIO1: U14.23 (GPIO1)
- new net ETH2_GPIO2: U14.24 (GPIO2)
- new net ETH2_GPIO3: U14.25 (RDY/GPIO3)
- new net ETH2_GPIO4: U14.32 (GPIO4)
- new net ETH2_GPIO5: U14.33 (GPIO5)
- new net ETH2_GPIO6: U14.34 (GPIO6)
- new net ETH2_GPIO7: U14.35 (GPIO7)
- new net ETH2_RST2: U14.26 (RST)
- new net ETH2_SEL: U14.27 (SEL)
Other:
- moved on the sheet: C10, C11, C34, C6, C7, T1, T2, T3, T4
