File: PSVB_EvalBoard/PSVB_EvalBoard.kicad_sch (KiCad schematic)
At the start: 454 parts, among them J1 PIN2, J10 PIN20, J11 PIN12_2x6, J12 PIN20, J13 PIN6_2x3, J29 PIN6_2x3, J3 PIN20, J30 PIN6_2x3, J31 PIN6_2x3, J4 PIN20, J5 PIN20, J6 PIN20, J7 PIN20, J8 PIN20, J9 PIN20, Q1 S9013, U1 SGM2036-ADJ, U12 STM32F429ZETx, U13 CH395Q, U14 CH395Q, U2 SGM2036-ADJ, U3 93LC56BT-IOT, U3 SGM2036-ADJ, U4 INA240A1PWR, U5 INA240A1PWR, U5 W25Q128JVSIQ, U6 24LC64ISN, U6 TM7707, U7 REF3030, U8 MPU6050, U8 REF3025, U9 REF3012, X1 2.4576Mhz, X2 12Mhz_Passive_3225, X3 16Mhz_Passive_3225, X4 30Mhz_3225, X5 30Mhz_3225

Commit message: updated PCB design-2023-5-24
Connections:
- net PG3: no longer J4.2
- net VSS: now also J4.2
Changed lines of the file:
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@@
     (stroke (width 0) (type default))
   )
+  (wire (pts (xy 293.37 408.94) (xy 309.88 408.94))
+    (stroke (width 0) (type default))
+  )
   (wire (pts (xy 443.23 72.39) (xy 481.33 72.39))
     (stroke (width 0) (type default))
@@
     (stroke (width 0) (type default))
   )
-  (wire (pts (xy 293.37 408.94) (xy 307.34 408.94))
-    (stroke (width 0) (type default))
-  )
   (wire (pts (xy 787.4 284.48) (xy 787.4 280.162))
     (stroke (width 0) (type default))
@@
     (effects (font (size 1.27 1.27) (thickness 0.254) bold (color 132 0 0 1)) (justify left bottom))
   )
-  (label "PG3" (at 303.53 408.94 0) (fields_autoplaced)
-    (effects (font (size 1.27 1.27)) (justify left bottom))
-  )
   (label "VCORE" (at 383.54 40.64 0) (fields_autoplaced)
     (effects (font (size 1.27 1.27)) (justify left bottom))
@@
         )
       )
+    )
+  )
+  (symbol (lib_id "power:VSS") (at 309.88 408.94 0) (unit 1)
+    (in_bom yes) (on_board yes) (dnp no)
+    (property "Reference" "#PWR0169" (at 309.88 412.75 0)
+      (effects (font (size 1.27 1.27)) hide)
+    )
+    (property "Value" "VSS" (at 309.88 405.13 0)
+      (effects (font (size 1.27 1.27)))
+    )
+    (property "Footprint" "" (at 309.88 408.94 0)
+      (effects (font (size 1.27 1.27)) hide)
+    )
+    (property "Datasheet" "" (at 309.88 408.94 0)
+      (effects (font (size 1.27 1.27)) hide)
+    )
+    (pin "1")
+    (instances
+      (project "PSVB_EvalBoard"
+        (path "/f2b0a56f-d786-40ff-9774-78e3f95871c8"
+          (reference "#PWR0169") (unit 1)
+        )
+      )

Commit message: almost finished the PCB design
Parts:
- removed R26: 0603 10K/1%, Resistor_SMD:R_0603_1608Metric_Pad0.98x0.95mm_HandSolder, symbol Device:R
Connections:
- net STM32_DAC_OUT0 is gone; now on net STM32_DAC_OUT1: R55.1
- net BTB_PB2: no longer J9.10
- net STM32_BOOT1: now also U12.48 (PB2)
- net STM32_DAC_OUT1: no longer R55.1
- net STM32_DAC_OUT2: now also R55.1
- net VSS: now also J5.10, J7.17, J7.19, J8.13, J8.15, J9.10
- removed net PB2: J5.10, U12.48 (PB2)

Commit message: 80 lines unconnected
Connections:
- net OPAMP1_IN: no longer J24.3
- net OPAMP1_IP: no longer J24.1
- net VSS: no longer J24.2
Other:
- moved on the sheet: J24
Changed lines of the file:
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@@
     (effects (font (size 1.27 1.27)) (justify left bottom))
   )
+  (label "PE5" (at 267.97 381 180) (fields_autoplaced)
+    (effects (font (size 1.27 1.27)) (justify right bottom))
+  )
   (label "PF4" (at 516.89 397.51 0) (fields_autoplaced)
     (effects (font (size 1.27 1.27)) (justify left bottom))
@@
     (effects (font (size 1.27 1.27)) (justify left bottom))
   )
-  (label "PE5" (at 264.16 381 0) (fields_autoplaced)
-    (effects (font (size 1.27 1.27)) (justify left bottom))
-  )
   (label "ETH2_TXD" (at 1068.07 741.68 0) (fields_autoplaced)
     (effects (font (size 1.27 1.27)) (justify left bottom))
@@
     )
   )
-  (symbol (lib_id "zgoolib:PIN3_1x3") (at 1148.08 474.98 0) (unit 1)
-    (in_bom yes) (on_board yes) (dnp no) (fields_autoplaced)
-    (property "Reference" "J24" (at 1154.43 475.615 0)
+  (symbol (lib_id "zgoolib:PIN3_1x3") (at 1148.08 474.98 0) (mirror y) (unit 1)
+    (in_bom yes) (on_board yes) (dnp no)
+    (property "Reference" "J24" (at 1141.73 475.615 0)
       (effects (font (size 1.27 1.27)) (justify left))
     )
-    (property "Value" "~" (at 1134.618 474.98 0)
+    (property "Value" "~" (at 1161.542 474.98 0)
       (effects (font (size 1.27 1.27)))
     )
@@
       (effects (font (size 1.27 1.27)) hide)
     )
-    (property "Datasheet" "" (at 1134.618 474.98 0)
+    (property "Datasheet" "" (at 1161.542 474.98 0)
       (effects (font (size 1.27 1.27)) hide)
     )

Commit message: Finished the PCB layout
Parts:
- added R42 (x4): 0603 1K/1%, Resistor_SMD:R_0603_1608Metric_Pad0.98x0.95mm_HandSolder, symbol Device:R
Changed lines of the file:
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@@
     )
   )
+  (symbol (lib_id "Device:R") (at 91.44 723.9 0) (unit 1)
+    (in_bom yes) (on_board yes) (dnp no)
+    (property "Reference" "R42" (at 88.9 728.98 90)
+      (effects (font (size 1.27 1.27)) (justify left))
+    )
+    (property "Value" "0603 1K/1%" (at 88.9 722.63 90)
+      (effects (font (size 1.27 1.27)) (justify left))
+    )
+    (property "Footprint" "Resistor_SMD:R_0603_1608Metric_Pad0.98x0.95mm_HandSolder" (at 89.662 723.9 90)
+      (effects (font (size 1.27 1.27)) hide)
+    )
+    (property "Datasheet" "~" (at 91.44 723.9 0)
+      (effects (font (size 1.27 1.27)) hide)
+    )
+    (pin "1")
+    (pin "2")
+    (instances
+      (project "PutuoEvalBoard_V2"
+        (path "/a62609cd-29b7-4918-b97d-7b2404ba61cf"
+          (reference "R42") (unit 1)
+        )
+      )
+      (project "PSVB_EvalBoard"
+        (path "/f2b0a56f-d786-40ff-9774-78e3f95871c8"
+          (reference "R159") (unit 1)
+        )
+      )
+    )
+  )
   (symbol (lib_id "Device:R") (at 326.39 207.01 0) (unit 1)
     (in_bom yes) (on_board yes) (dnp no)
@@
     )
   )
+  (symbol (lib_id "Device:R") (at 100.33 723.9 0) (unit 1)
+    (in_bom yes) (on_board yes) (dnp no)
+    (property "Reference" "R42" (at 97.79 728.98 90)
+      (effects (font (size 1.27 1.27)) (justify left))
+    )
+    (property "Value" "0603 1K/1%" (at 97.79 722.63 90)
+      (effects (font (size 1.27 1.27)) (justify left))
+    )
+    (property "Footprint" "Resistor_SMD:R_0603_1608Metric_Pad0.98x0.95mm_HandSolder" (at 98.552 723.9 90)
+      (effects (font (size 1.27 1.27)) hide)
+    )
+    (property "Datasheet" "~" (at 100.33 723.9 0)
+      (effects (font (size 1.27 1.27)) hide)
+    )
+    (pin "1")
+    (pin "2")
+    (instances
+      (project "PutuoEvalBoard_V2"
+        (path "/a62609cd-29b7-4918-b97d-7b2404ba61cf"
+          (reference "R42") (unit 1)
+        )
+      )
+      (project "PSVB_EvalBoard"
+        (path "/f2b0a56f-d786-40ff-9774-78e3f95871c8"
+          (reference "R163") (unit 1)
+        )
+      )
+    )
+  )
   (symbol (lib_id "power:+5V") (at 151.13 43.18 0) (unit 1)
     (in_bom yes) (on_board yes) (dnp no)
@@
     )
   )
+  (symbol (lib_id "Device:R") (at 82.55 723.9 0) (unit 1)
+    (in_bom yes) (on_board yes) (dnp no)
+    (property "Reference" "R42" (at 80.01 728.98 90)
+      (effects (font (size 1.27 1.27)) (justify left))
+    )
+    (property "Value" "0603 1K/1%" (at 80.01 722.63 90)
+      (effects (font (size 1.27 1.27)) (justify left))
+    )
+    (property "Footprint" "Resistor_SMD:R_0603_1608Metric_Pad0.98x0.95mm_HandSolder" (at 80.772 723.9 90)
+      (effects (font (size 1.27 1.27)) hide)
+    )
+    (property "Datasheet" "~" (at 82.55 723.9 0)
+      (effects (font (size 1.27 1.27)) hide)
+    )
+    (pin "1")
+    (pin "2")
+    (instances
+      (project "PutuoEvalBoard_V2"
+        (path "/a62609cd-29b7-4918-b97d-7b2404ba61cf"
+          (reference "R42") (unit 1)
+        )
+      )
+      (project "PSVB_EvalBoard"
+        (path "/f2b0a56f-d786-40ff-9774-78e3f95871c8"
+          (reference "R158") (unit 1)
+        )
+      )
+    )
+  )
   (symbol (lib_id "zgoolib:PIN6_1x6") (at 1145.54 368.935 0) (unit 1)
     (in_bom yes) (on_board yes) (dnp no)
@@
         )
       )
+    )
+  )
+  (symbol (lib_id "Device:R") (at 109.22 723.9 0) (unit 1)
+    (in_bom yes) (on_board yes) (dnp no)
+    (property "Reference" "R42" (at 106.68 728.98 90)
+      (effects (font (size 1.27 1.27)) (justify left))
+    )
+    (property "Value" "0603 1K/1%" (at 106.68 722.63 90)
+      (effects (font (size 1.27 1.27)) (justify left))
+    )
+    (property "Footprint" "Resistor_SMD:R_0603_1608Metric_Pad0.98x0.95mm_HandSolder" (at 107.442 723.9 90)
+      (effects (font (size 1.27 1.27)) hide)
+    )
+    (property "Datasheet" "~" (at 109.22 723.9 0)
+      (effects (font (size 1.27 1.27)) hide)
+    )
+    (pin "1")
+    (pin "2")
+    (instances
+      (project "PutuoEvalBoard_V2"
+        (path "/a62609cd-29b7-4918-b97d-7b2404ba61cf"
+          (reference "R42") (unit 1)
+        )
+      )
+      (project "PSVB_EvalBoard"
+        (path "/f2b0a56f-d786-40ff-9774-78e3f95871c8"
+          (reference "R182") (unit 1)
+        )
+      )
