File: PSVB_EvalBoard/PSVB_EvalBoard.kicad_sch (KiCad schematic)
At the start: 457 parts, among them J1 PIN2, J10 PIN20, J11 PIN12_2x6, J12 PIN20, J13 PIN6_2x3, J29 PIN6_2x3, J3 PIN20, J30 PIN6_2x3, J31 PIN6_2x3, J4 PIN20, J5 PIN20, J6 PIN20, J7 PIN20, J8 PIN20, J9 PIN20, Q1 S9013, U1 SGM2036-ADJ, U12 STM32F429ZETx, U13 CH395Q, U14 CH395Q, U2 SGM2036-ADJ, U3 93LC56BT-IOT, U3 SGM2036-ADJ, U4 INA240A1PWR, U5 INA240A1PWR, U5 W25Q128JVSIQ, U6 24LC64ISN, U6 TM7707, U7 REF3030, U8 MPU6050, U8 REF3025, U9 REF3012, X1 2.4576Mhz, X2 12Mhz_Passive_3225, X3 16Mhz_Passive_3225, X4 30Mhz_3225, X5 30Mhz_3225

Commit message: Did some modification.
Parts:
- added R42: 0603 1K/1%, Resistor_SMD:R_0603_1608Metric_Pad0.98x0.95mm_HandSolder, symbol Device:R
Other:
- moved on the sheet: R42
Changed lines of the file:
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@@
     )
   )
-  (symbol (lib_id "Device:R") (at 91.44 723.9 0) (unit 1)
+  (symbol (lib_id "Device:R") (at 86.36 721.36 0) (unit 1)
     (in_bom yes) (on_board yes) (dnp no)
-    (property "Reference" "R42" (at 88.9 728.98 90)
+    (property "Reference" "R42" (at 83.82 728.98 90)
       (effects (font (size 1.27 1.27)) (justify left))
     )
-    (property "Value" "0603 1K/1%" (at 88.9 722.63 90)
+    (property "Value" "0603 1K/1%" (at 83.82 721.36 90)
       (effects (font (size 1.27 1.27)) (justify left))
     )
-    (property "Footprint" "Resistor_SMD:R_0603_1608Metric_Pad0.98x0.95mm_HandSolder" (at 89.662 723.9 90)
+    (property "Footprint" "Resistor_SMD:R_0603_1608Metric_Pad0.98x0.95mm_HandSolder" (at 84.582 721.36 90)
       (effects (font (size 1.27 1.27)) hide)
     )
-    (property "Datasheet" "~" (at 91.44 723.9 0)
+    (property "Datasheet" "~" (at 86.36 721.36 0)
       (effects (font (size 1.27 1.27)) hide)
     )
@@
     )
   )
-  (symbol (lib_id "Device:R") (at 100.33 723.9 0) (unit 1)
+  (symbol (lib_id "Device:R") (at 92.71 721.36 0) (unit 1)
     (in_bom yes) (on_board yes) (dnp no)
-    (property "Reference" "R42" (at 97.79 728.98 90)
+    (property "Reference" "R42" (at 90.17 728.98 90)
       (effects (font (size 1.27 1.27)) (justify left))
     )
-    (property "Value" "0603 1K/1%" (at 97.79 722.63 90)
+    (property "Value" "0603 1K/1%" (at 90.17 721.36 90)
       (effects (font (size 1.27 1.27)) (justify left))
     )
-    (property "Footprint" "Resistor_SMD:R_0603_1608Metric_Pad0.98x0.95mm_HandSolder" (at 98.552 723.9 90)
+    (property "Footprint" "Resistor_SMD:R_0603_1608Metric_Pad0.98x0.95mm_HandSolder" (at 90.932 721.36 90)
       (effects (font (size 1.27 1.27)) hide)
     )
-    (property "Datasheet" "~" (at 100.33 723.9 0)
+    (property "Datasheet" "~" (at 92.71 721.36 0)
       (effects (font (size 1.27 1.27)) hide)
     )
@@
     )
   )
-  (symbol (lib_id "Device:R") (at 82.55 723.9 0) (unit 1)
+  (symbol (lib_id "Device:R") (at 80.01 721.36 0) (unit 1)
     (in_bom yes) (on_board yes) (dnp no)
-    (property "Reference" "R42" (at 80.01 728.98 90)
+    (property "Reference" "R42" (at 77.47 728.98 90)
       (effects (font (size 1.27 1.27)) (justify left))
     )
-    (property "Value" "0603 1K/1%" (at 80.01 722.63 90)
+    (property "Value" "0603 1K/1%" (at 77.47 721.36 90)
       (effects (font (size 1.27 1.27)) (justify left))
     )
-    (property "Footprint" "Resistor_SMD:R_0603_1608Metric_Pad0.98x0.95mm_HandSolder" (at 80.772 723.9 90)
+    (property "Footprint" "Resistor_SMD:R_0603_1608Metric_Pad0.98x0.95mm_HandSolder" (at 78.232 721.36 90)
       (effects (font (size 1.27 1.27)) hide)
     )
-    (property "Datasheet" "~" (at 82.55 723.9 0)
+    (property "Datasheet" "~" (at 80.01 721.36 0)
       (effects (font (size 1.27 1.27)) hide)
     )
@@
     )
   )
+  (symbol (lib_id "Device:R") (at 105.41 721.36 0) (unit 1)
+    (in_bom yes) (on_board yes) (dnp no)
+    (property "Reference" "R42" (at 102.87 728.98 90)
+      (effects (font (size 1.27 1.27)) (justify left))
+    )
+    (property "Value" "0603 1K/1%" (at 102.87 721.36 90)
+      (effects (font (size 1.27 1.27)) (justify left))
+    )
+    (property "Footprint" "Resistor_SMD:R_0603_1608Metric_Pad0.98x0.95mm_HandSolder" (at 103.632 721.36 90)
+      (effects (font (size 1.27 1.27)) hide)
+    )
+    (property "Datasheet" "~" (at 105.41 721.36 0)
+      (effects (font (size 1.27 1.27)) hide)
+    )
+    (pin "1")
+    (pin "2")
+    (instances
+      (project "PutuoEvalBoard_V2"
+        (path "/a62609cd-29b7-4918-b97d-7b2404ba61cf"
+          (reference "R42") (unit 1)
+        )
+      )
+      (project "PSVB_EvalBoard"
+        (path "/f2b0a56f-d786-40ff-9774-78e3f95871c8"
+          (reference "R198") (unit 1)
+        )
+      )
+    )
+  )
   (symbol (lib_id "power:VSS") (at 915.67 344.17 180) (unit 1)
     (in_bom yes) (on_board yes) (dnp no)
@@
     )
   )
-  (symbol (lib_id "Device:R") (at 109.22 723.9 0) (unit 1)
+  (symbol (lib_id "Device:R") (at 99.06 721.36 0) (unit 1)
     (in_bom yes) (on_board yes) (dnp no)
-    (property "Reference" "R42" (at 106.68 728.98 90)
+    (property "Reference" "R42" (at 96.52 728.98 90)
       (effects (font (size 1.27 1.27)) (justify left))
     )
-    (property "Value" "0603 1K/1%" (at 106.68 722.63 90)
+    (property "Value" "0603 1K/1%" (at 96.52 721.36 90)
       (effects (font (size 1.27 1.27)) (justify left))
     )
-    (property "Footprint" "Resistor_SMD:R_0603_1608Metric_Pad0.98x0.95mm_HandSolder" (at 107.442 723.9 90)
+    (property "Footprint" "Resistor_SMD:R_0603_1608Metric_Pad0.98x0.95mm_HandSolder" (at 97.282 721.36 90)
       (effects (font (size 1.27 1.27)) hide)
     )
-    (property "Datasheet" "~" (at 109.22 723.9 0)
+    (property "Datasheet" "~" (at 99.06 721.36 0)
       (effects (font (size 1.27 1.27)) hide)
     )
