File: PSVB_EvalBoard/_autosave-PSVB_EvalBoard.kicad_sch (KiCad schematic)
At the start: 458 parts, among them J1 PIN2, J10 PIN20, J11 PIN12_2x6, J12 PIN20, J13 PIN6_2x3, J29 PIN6_2x3, J3 PIN20, J30 PIN6_2x3, J31 PIN6_2x3, J4 PIN20, J5 PIN20, J6 PIN20, J7 PIN20, J8 PIN20, J9 PIN20, Q1 S9013, U1 SGM2036-ADJ, U12 STM32F429ZETx, U13 CH395Q, U14 CH395Q, U16 MPU6050, U2 SGM2036-ADJ, U3 93LC56BT-IOT, U3 SGM2036-ADJ, U4 INA240A1PWR, U5 INA240A1PWR, U5 W25Q128JVSIQ, U6 24LC64ISN, U6 TM7707, U7 REF3030, U8 REF3025, U9 REF3012, X1 2.4576Mhz, X2 12Mhz_Passive_3225, X3 16Mhz_Passive_3225, X4 30Mhz_3225, X5 30Mhz_3225

Commit message: Fixed some issues.
Connections:
- net PF9 is gone; now on net STM32_USB_ID: J3.16
Changed lines of the file:
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@@
-    (effects (font (size 1.27 1.27)) (justify left bottom))
-  )
-  (label "PF9" (at 303.53 391.16 0) (fields_autoplaced)
     (effects (font (size 1.27 1.27)) (justify left bottom))
   )
@@
     (effects (font (size 1.27 1.27)) (justify left bottom))
   )
+  (label "STM32_USB_ID" (at 294.005 391.16 0) (fields_autoplaced)
+    (effects (font (size 1.27 1.27) (color 255 0 0 1)) (justify left bottom))
+  )
   (label "AKINA_JTDO" (at 693.42 306.07 0) (fields_autoplaced)

Commit message: Finished PCB layout.
Parts:
- added R42: 0603 47K/1%, Resistor_SMD:R_0603_1608Metric_Pad0.98x0.95mm_HandSolder, symbol Device:R
- R42: value 0603 1K/1% -> 0603 47K/1%
Connections:
- net +3V3: now also R42.2, R42.2, R42.2, R42.2, R42.2, R42.2
- net BTB_PB2: now also J9.10
- net OPAMP1_IN: now also J24.3
- net OPAMP1_IP: now also J24.1
- net PC10: now also R42.1
- net PC11: now also R42.1
- net PC8: now also R42.1
- net PC9: now also R42.1
- net PD2: now also R42.1
- net PD3: now also R42.1
- net VSS: now also BTB100x1.69, J24.2; no longer J9.10
Other:
- moved on the sheet: J24, R42, SD1
